File: Zynq-eame_UltraScale_0/KiCad/MIO&REFERENCE.sch (KiCad schematic (older format))
At the start: 42 parts, among them J1 USB_B_Micro, J2 Conn_01x06, SW1 SW_Push, U1 XCZU2CG, U3 FT2232H, U4 93C46, Y1 12MHz

Commit message: upd
Parts:
- added C? (x3): 100nF, Capacitor_SMD:C_0805_2012Metric, symbol Device:C
- added J?: Micro_SD_Card, symbol Connector:Micro_SD_Card
- added R?: 330, Resistor_SMD:R_0805_2012Metric, symbol Device:R
- added R?: 4.7K, Resistor_SMD:R_0805_2012Metric, symbol Device:R
- added U?: MT25QU512ABB, Zynq-eame_UltraScale_0:BGA-25_5x5_6.0x8.0mm, symbol Zynq_UltraScale:MT25QU512ABB
- added U?: IP4856CX25, Zynq-eame_UltraScale_0:BGA-25_5x5_2.049999x2.049999mm, symbol Zynq_UltraScale:IP4856CX25
- R9, R?: value R -> 10k; footprint (none) -> Resistor_SMD:R_0805_2012Metric
- R?: value R -> 820; footprint (none) -> Resistor_SMD:R_0805_2012Metric
- R?: value R -> 1300; footprint (none) -> Resistor_SMD:R_0805_2012Metric
Connections:
- net +1V8: now also C?.1, C?.1, R?.1, U?.B3 (VCCA), U?.B4 (VCC)
- net +3V3: now also C?.1, J?.4 (VDD), R?.2, U?.A4 (VSUPPLY), U?.C4 (V_SD_REF)
- net GND: now also C?.2, C?.2, C?.2, J?.6 (VSS), J?.9 (SHIELD), U?.B3 (VSS), U?.C3 (GND)
- net QSPI_CS: now reaches U1.AA1 (PS_MIO5)
- net QSPI_CS: now also R?.2, U?.C2 (S#)
- net QSPI_CLK: now reaches U1.U4 (PS_MIO0)
- net QSPI_CLK: now also U?.B2 (C)
- net QSPI_DQ3: now reaches U1.U5 (PS_MIO3)
- net QSPI_DQ3: now also U?.D4 (DQ3)
- net QSPI_DQ0: now reaches U1.U6 (PS_MIO4)
- net QSPI_DQ0: now also U?.D3 (DQ0)
- net QSPI_DQ2: now reaches U1.V2 (PS_MIO2)
- net QSPI_DQ2: now also U?.C4 (W#/DQ2)
- net QSPI_DQ1: now reaches U1.W1 (PS_MIO1)
- net QSPI_DQ1: now also U?.D2 (DQ1)
- net MIO_SD1_DAT3: now reaches U1.A12 (PS_MIO48)
- net MIO_SD1_DAT3: now also U?.B1 (DATA3_H)
- net MIO_SD1_CMD: now reaches U1.A13 (PS_MIO50)
- net MIO_SD1_CMD: now also U?.D2 (CMD_H)
- net MIO_SD1_DIR_DAT0: now reaches U1.B10 (PS_MIO41)
- net MIO_SD1_DIR_DAT0: now also U?.A3 (DIR_0)
- net MIO_SD1_DAT1: now reaches U1.B12 (PS_MIO47)
- net MIO_SD1_DAT1: now also U?.E1 (DATA1_H)
- net MIO_SD1_DAT0: now reaches U1.C12 (PS_MIO46)
- net MIO_SD1_DAT0: now also U?.D1 (DATA0_H)
- net MIO_SD1_CLK: now reaches U1.C13 (PS_MIO51)
- net MIO_SD1_CLK: now also U?.C1 (CLK_IN)
- net MIO_SD1_DIR_CMD: now reaches U1.D11 (PS_MIO40)
- net MIO_SD1_DIR_CMD: now also U?.A2 (DIR_CMD)
- net MIO_SD1_DAT2: now reaches U1.D13 (PS_MIO49)
- net MIO_SD1_DAT2: now also U?.A1 (DATA2_H)
- new net: U?.A2 (NC), U?.A3 (RFU), U?.A4 (RESET#), U?.A4Ç (RFU), U?.A5 (RFU), U?.B1 (RFU), U?.B5 (RFU), U?.C1 (RFU), U?.C3 (RFU), U?.C5 (RFU), U?.D1 (RFU), U?.D5 (RFU), U?.E1 (RFU), U?.E2 (RFU), U?.E3 (RFU), U?.E5 (RFU)
- new net: R?.1, U?.C2 (ENABLE)
- new net MIO_SD1_DIR_DAT1: U?.E3 (DIR_1_3)
- new net MIO_SD1_SEL: U?.B2 (SEL)
- new net SD_CLK: J?.5 (CLK), U?.C5 (CLK_SD)
- new net SD_CMD: J?.3 (CMD), U?.C4 (V_SD_REF)
- new net SD_DAT0: J?.7 (DAT0), U?.D5 (DATA0_SD)
- new net SD_DAT1: J?.8 (DAT1), U?.E5 (DATA1_SD)
- new net SD_DAT2: J?.1 (DAT2), U?.A5 (DATA2_SD)
- new net SD_DAT3: J?.2 (DAT3/CD), U?.B5 (DATA3_SD)
- no-connect marks 38 -> 41
Other:
- note added: "BOOT RST\n\n"
- note added: "QUAD-SPI \nFLASH MEMORY"
- note added: "SD CONNECTOR"
- moved on the sheet: D1, D?, R1, R2, R3, R4, R7, R?, SW1

Commit message: UPD
Parts:
- added C18, C?: 100nF, Capacitor_SMD:C_0805_2012Metric, symbol Device:C
- added C?: 4.7uF, Capacitor_SMD:C_0805_2012Metric, symbol Device:C
- added J?: USB_B_Micro, symbol Connector:USB_B_Micro
- added R19: 4.7K, Resistor_SMD:R_0805_2012Metric, symbol Device:R
- added R?: 1k, Resistor_SMD:R_0805_2012Metric, symbol Device:R
- added R?: 4.7k, Resistor_SMD:R_0805_2012Metric, symbol Device:R
- added R?: 10k, Resistor_SMD:R_0805_2012Metric, symbol Device:R
- added U?: XCZU2CG, Zynq-eame_UltraScale_0:SBVA484, symbol Zynq_UltraScale:XCZU2CG
- added U?: CP2102N-A01-GQFN28, Package_DFN_QFN:QFN-28-1EP_5x5mm_P0.5mm_EP3.35x3.35mm, symbol Interface_USB:CP2102N-A01-GQFN28
- added X1: ASE-33.333MHz, Oscillator:Oscillator_SMD_Abracon_ASE-4Pin_3.2x2.5mm, symbol Oscillator:ASE-xxxMHz
- gave numbers to parts that had none: 15
Connections:
- net +3V3: now also C18.2, R19.1, X1.4 (Vdd)
- net GND: now also C18.1, C?.1, C?.2, J?.5 (GND), J?.6 (Shield), R?.2, U?.29 (GND), U?.3 (GND), X1.2 (GND)
- net PS_CLK: now also X1.3 (OUT)
- net MIO8_TX: now reaches U1.V3 (PS_MIO8)
- net MIO8_TX: now also U?.25 (RXD)
- net MIO9_RX: now reaches U1.V5 (PS_MIO9)
- net MIO9_RX: now also U?.26 (TXD)
- new net: R19.2, X1.1 (EN)
- new net: J?.3 (D+), U?.4 (D+)
- new net: J?.2 (D-), U?.5 (D-)
- new net: C?.1, R?.1, U?.6 (VDD)
- new net: C?.2, J?.1 (VBUS), R?.2, U?.7 (REGIN)
- new net: R?.1, R?.1, U?.8 (VBUS)
- new net: R?.2, U?.9 (~RSTb)
- no-connect marks 41 -> 145
Other:
- note added: "OSCILLATOR 33MHz"
- note added: "USB-UART"

Commit message: upd
Connections:
- no-connect marks 145 -> 146
Changed lines of the file:
@@
 Wire Wire Line
 	9500 2100 9850 2100
+NoConn ~ 8750 6800
 $EndSCHEMATC

Commit message: upd
Parts:
- gave numbers to parts that had none: 8
Changed lines of the file:
@@
 	9550 10350 9200 10350
 $Comp
-L Zynq_UltraScale:XCZU2CG U?
+L Zynq_UltraScale:XCZU2CG U1
 U 10 1 602B7019
 P 13250 8200
-F 0 "U?" H 13258 9765 50  0000 C CNN
+F 0 "U1" H 13258 9765 50  0000 C CNN
 F 1 "XCZU2CG" H 13258 9674 50  0000 C CNN
 F 2 "Zynq-eame_UltraScale_0:SBVA484" H 13150 3450 50  0001 C CNN
@@
 NoConn ~ 13600 3700
 $Comp
-L Interface_USB:CP2102N-A01-GQFN28 U?
+L Interface_USB:CP2102N-A01-GQFN28 U12
 U 1 1 605EF620
 P 10100 7200
-F 0 "U?" H 9750 8450 50  0000 C CNN
+F 0 "U12" H 9750 8450 50  0000 C CNN
 F 1 "CP2102N-A01-GQFN28" H 10600 5950 50  0000 C CNN
 F 2 "Package_DFN_QFN:QFN-28-1EP_5x5mm_P0.5mm_EP3.35x3.35mm" H 10550 6000 50  0001 L CNN
@@
 $EndComp
 $Comp
-L Connector:USB_B_Micro J?
+L Connector:USB_B_Micro J5
 U 1 1 60605CEA
 P 8450 6600
-F 0 "J?" H 8507 7067 50  0000 C CNN
+F 0 "J5" H 8507 7067 50  0000 C CNN
 F 1 "USB_B_Micro" H 8507 6976 50  0000 C CNN
 F 2 "" H 8600 6550 50  0001 C CNN
@@
 	8750 6700 9600 6700
 $Comp
-L Device:R R?
+L Device:R R63
 U 1 1 6065D8D6
 P 9500 6100
-F 0 "R?" H 9570 6146 50  0000 L CNN
+F 0 "R63" H 9570 6146 50  0000 L CNN
 F 1 "1k" H 9570 6055 50  0000 L CNN
 F 2 "Resistor_SMD:R_0805_2012Metric" V 9430 6100 50  0001 C CNN
@@
 $EndComp
 $Comp
-L Device:R R?
+L Device:R R61
 U 1 1 6065F94D
 P 9200 6400
-F 0 "R?" V 8993 6400 50  0000 C CNN
+F 0 "R61" V 8993 6400 50  0000 C CNN
 F 1 "4.7k" V 9084 6400 50  0000 C CNN
 F 2 "Resistor_SMD:R_0805_2012Metric" V 9130 6400 50  0001 C CNN
@@
 $EndComp
 $Comp
-L Device:R R?
+L Device:R R62
 U 1 1 6066177E
 P 9450 7000
-F 0 "R?" H 9520 7046 50  0000 L CNN
+F 0 "R62" H 9520 7046 50  0000 L CNN
 F 1 "10k" H 9520 6955 50  0000 L CNN
 F 2 "Resistor_SMD:R_0805_2012Metric" V 9380 7000 50  0001 C CNN
@@
 $EndComp
 $Comp
-L power:GND #PWR?
+L power:GND #PWR0245
 U 1 1 60663506
 P 9450 7300
-F 0 "#PWR?" H 9450 7050 50  0001 C CNN
+F 0 "#PWR0245" H 9450 7050 50  0001 C CNN
 F 1 "GND" H 9455 7127 50  0000 C CNN
 F 2 "" H 9450 7300 50  0001 C CNN
@@
 $EndComp
 $Comp
-L power:GND #PWR?
+L power:GND #PWR0246
 U 1 1 60665452
 P 10100 8650
-F 0 "#PWR?" H 10100 8400 50  0001 C CNN
+F 0 "#PWR0246" H 10100 8400 50  0001 C CNN
 F 1 "GND" H 10105 8477 50  0000 C CNN
 F 2 "" H 10100 8650 50  0001 C CNN
@@
 $EndComp
 $Comp
-L power:GND #PWR?
+L power:GND #PWR0247
 U 1 1 606675EF
 P 8450 7150
-F 0 "#PWR?" H 8450 6900 50  0001 C CNN
+F 0 "#PWR0247" H 8450 6900 50  0001 C CNN
 F 1 "GND" H 8455 6977 50  0000 C CNN
 F 2 "" H 8450 7150 50  0001 C CNN
@@
 $EndComp
 $Comp
-L Device:C C?
+L Device:C C35
 U 1 1 6066B14D
 P 8900 6050
-F 0 "C?" H 8900 6150 50  0000 L CNN
+F 0 "C35" H 8900 6150 50  0000 L CNN
 F 1 "4.7uF" H 8600 6150 50  0000 L CNN
 F 2 "Capacitor_SMD:C_0805_2012Metric" H 8938 5900 50  0001 C CNN
@@
 Connection ~ 9050 6400
 $Comp
-L power:GND #PWR?
+L power:GND #PWR0248
 U 1 1 6074D221
 P 8900 5800
-F 0 "#PWR?" H 8900 5550 50  0001 C CNN
+F 0 "#PWR0248" H 8900 5550 50  0001 C CNN
 F 1 "GND" H 8905 5627 50  0000 C CNN
 F 2 "" H 8900 5800 50  0001 C CNN
@@
 $EndComp
 $Comp
-L power:GND #PWR?
+L power:GND #PWR0249
 U 1 1 60762EEE
 P 10550 5800
-F 0 "#PWR?" H 10550 5550 50  0001 C CNN
+F 0 "#PWR0249" H 10550 5550 50  0001 C CNN
 F 1 "GND" H 10555 5627 50  0000 C CNN
 F 2 "" H 10550 5800 50  0001 C CNN
@@
 $EndComp
 $Comp
-L Device:C C?
+L Device:C C36
 U 1 1 60778C2C
 P 10350 5800
-F 0 "C?" V 10500 5850 50  0000 L CNN
+F 0 "C36" V 10500 5850 50  0000 L CNN
 F 1 "100nF" V 10500 5500 50  0000 L CNN
 F 2 "Capacitor_SMD:C_0805_2012Metric" H 10388 5650 50  0001 C CNN
