File: Zynq-eame_UltraScale_0/KiCad/PINOUT.sch (KiCad schematic (older format))
At the start: 3 parts

Commit message: UPD
Parts:
- added D? (x5): LED_ALT, symbol Device:LED_ALT
- added Q? (x5): MMBF170, Package_TO_SOT_SMD:SOT-23, symbol Transistor_FET:MMBF170
- added R? (x15): 4.7K, Resistor_SMD:R_0805_2012Metric, symbol Device:R
- added R? (x5): 10K, Resistor_SMD:R_0805_2012Metric, symbol Device:R
- added R? (x5): 1K, Resistor_SMD:R_0805_2012Metric, symbol Device:R
- added SW? (x5): SW_SPST, Button_Switch_SMD:SW_DIP_SPSTx01_Slide_6.7x4.1mm_W6.73mm_P2.54mm_LowProfile_JPin, symbol Switch:SW_SPST
- added SW? (x5): SW_Push, symbol Switch:SW_Push
- gave numbers to parts that had none: 1
Connections:
- net BT_1: now reaches U1.F4 (IO_T3U_N12_65)
- net BT_1: now also R?.2, SW?.1
- net BT_5: now reaches U1.G2 (IO_L17N_T2U_N9_AD10N_65)
- net BT_5: now also R?.2, SW?.1
- net BT_3: now reaches U1.G4 (IO_L18N_T2U_N11_AD2N_65)
- net BT_3: now also R?.2, SW?.1
- net SW_1: now reaches U1.H2 (IO_L17P_T2U_N8_AD10P_65)
- net SW_1: now also R?.2, SW?.1 (A)
- net BT_2: now reaches U1.H3 (IO_T2U_N12_65)
- net BT_2: now also R?.2, SW?.1
- net BT_4: now reaches U1.H4 (IO_L18P_T2U_N10_AD2P_65)
- net BT_4: now also R?.2, SW?.1
- net SW_2: now reaches U1.H5 (IO_L16N_T2U_N7_QBC_AD3N_65)
- net SW_2: now also R?.2, SW?.1 (A)
- net SW_4: now reaches U1.J1 (IO_L15N_T2L_N5_AD11N_65)
- net SW_4: now also R?.2, SW?.1 (A)
- net LED_3: now reaches U1.J2 (IO_L13N_T2L_N1_GC_QBC_65)
- net LED_3: now also R?.2
- net LED_4: now reaches U1.J3 (IO_L13P_T2L_N0_GC_QBC_65)
- net LED_4: now also R?.2
- net SW_3: now reaches U1.J5 (IO_L16P_T2U_N6_QBC_AD3P_65)
- net SW_3: now also R?.2, SW?.1 (A)
- net SW_5: now reaches U1.K1 (IO_L15P_T2L_N4_AD11P_65)
- net SW_5: now also R?.2, SW?.1 (A)
- net LED_1: now reaches U1.K3 (IO_L14N_T2L_N3_GC_65)
- net LED_1: now also R?.2
- net LED_2: now reaches U1.K4 (IO_L14P_T2L_N2_GC_65)
- net LED_2: now also R?.2
- net LED_5: now reaches U1.L3 (IO_L12N_T1U_N11_GC_65)
- net LED_5: now also R?.2
- new net: D?.1 (K), R?.1 (x5)
- new net: Q?.3 (D), R?.2 (x5)
- new net: Q?.1 (G), R?.1, R?.1 (x5)
- new net +3V3: D?.2 (A), D?.2 (A), D?.2 (A), D?.2 (A), D?.2 (A), R?.1, R?.1, R?.1, R?.1, R?.1, SW?.2, SW?.2, SW?.2, SW?.2, SW?.2
- new net GND: Q?.2 (S), Q?.2 (S), Q?.2 (S), Q?.2 (S), Q?.2 (S), R?.1, R?.1, R?.1, R?.1, R?.1, R?.2, R?.2, R?.2, R?.2, R?.2, SW?.2 (B), SW?.2 (B), SW?.2 (B), SW?.2 (B), SW?.2 (B)
- no-connect marks 4 -> 67
Other:
- note added: "BUTTONS\n\n"
- note added: "LEDS\n"
- note added: "SWITCHES\n"
- moved on the sheet: U1B, U1C, U1D

Commit message: upd
Connections:
- net +3V3: no longer R?.1, R?.1, R?.1, R?.1, R?.1, SW?.2, SW?.2, SW?.2, SW?.2, SW?.2
- new net +1V8: R?.1, R?.1, R?.1, R?.1, R?.1, SW?.2, SW?.2, SW?.2, SW?.2, SW?.2
Changed lines of the file:
@@
-$EndComp
-$Comp
-L power:+3.3V #PWR?
-U 1 1 604FEBB4
-P 9100 5550
-F 0 "#PWR?" H 9100 5400 50  0001 C CNN
-F 1 "+3.3V" H 9115 5723 50  0000 C CNN
-F 2 "" H 9100 5550 50  0001 C CNN
-F 3 "" H 9100 5550 50  0001 C CNN
-	1    9100 5550
-	1    0    0    -1
 $EndComp
 $Comp
@@
 $EndComp
 $Comp
-L power:+3.3V #PWR?
-U 1 1 60505BE4
-P 9700 5550
-F 0 "#PWR?" H 9700 5400 50  0001 C CNN
-F 1 "+3.3V" H 9715 5723 50  0000 C CNN
-F 2 "" H 9700 5550 50  0001 C CNN
-F 3 "" H 9700 5550 50  0001 C CNN
-	1    9700 5550
-	1    0    0    -1
-$EndComp
-$Comp
 L power:GND #PWR?
 U 1 1 60505BEA
@@
 $EndComp
 $Comp
-L power:+3.3V #PWR?
-U 1 1 60506FB1
-P 10250 5550
-F 0 "#PWR?" H 10250 5400 50  0001 C CNN
-F 1 "+3.3V" H 10265 5723 50  0000 C CNN
-F 2 "" H 10250 5550 50  0001 C CNN
-F 3 "" H 10250 5550 50  0001 C CNN
-	1    10250 5550
-	1    0    0    -1
-$EndComp
-$Comp
 L power:GND #PWR?
 U 1 1 60506FB7
@@
 $EndComp
 $Comp
-L power:+3.3V #PWR?
-U 1 1 60507FC1
-P 10800 5550
-F 0 "#PWR?" H 10800 5400 50  0001 C CNN
-F 1 "+3.3V" H 10815 5723 50  0000 C CNN
-F 2 "" H 10800 5550 50  0001 C CNN
-F 3 "" H 10800 5550 50  0001 C CNN
-	1    10800 5550
-	1    0    0    -1
-$EndComp
-$Comp
 L power:GND #PWR?
 U 1 1 60507FC7
@@
 $EndComp
 $Comp
-L power:+3.3V #PWR?
-U 1 1 605094AE
-P 11350 5550
-F 0 "#PWR?" H 11350 5400 50  0001 C CNN
-F 1 "+3.3V" H 11365 5723 50  0000 C CNN
-F 2 "" H 11350 5550 50  0001 C CNN
-F 3 "" H 11350 5550 50  0001 C CNN
-	1    11350 5550
-	1    0    0    -1
-$EndComp
-$Comp
 L power:GND #PWR?
 U 1 1 605094B4
@@
 	1    12900 6400
 	1    0    0    1
-$EndComp
-$Comp
-L power:+3.3V #PWR?
-U 1 1 6050AEDB
-P 12900 5550
-F 0 "#PWR?" H 12900 5400 50  0001 C CNN
-F 1 "+3.3V" H 12915 5723 50  0000 C CNN
-F 2 "" H 12900 5550 50  0001 C CNN
-F 3 "" H 12900 5550 50  0001 C CNN
-	1    12900 5550
-	1    0    0    -1
 $EndComp
 $Comp
@@
 $EndComp
 $Comp
-L power:+3.3V #PWR?
-U 1 1 60511FAF
-P 13450 5550
-F 0 "#PWR?" H 13450 5400 50  0001 C CNN
-F 1 "+3.3V" H 13465 5723 50  0000 C CNN
-F 2 "" H 13450 5550 50  0001 C CNN
-F 3 "" H 13450 5550 50  0001 C CNN
-	1    13450 5550
-	1    0    0    -1
-$EndComp
-$Comp
 L power:GND #PWR?
 U 1 1 60511FB5
@@
 $EndComp
 $Comp
-L power:+3.3V #PWR?
-U 1 1 60512FB4
-P 14000 5550
-F 0 "#PWR?" H 14000 5400 50  0001 C CNN
-F 1 "+3.3V" H 14015 5723 50  0000 C CNN
-F 2 "" H 14000 5550 50  0001 C CNN
-F 3 "" H 14000 5550 50  0001 C CNN
-	1    14000 5550
-	1    0    0    -1
-$EndComp
-$Comp
 L power:GND #PWR?
 U 1 1 60512FBA
@@
 $EndComp
 $Comp
-L power:+3.3V #PWR?
-U 1 1 6051419F
-P 14550 5550
-F 0 "#PWR?" H 14550 5400 50  0001 C CNN
-F 1 "+3.3V" H 14565 5723 50  0000 C CNN
-F 2 "" H 14550 5550 50  0001 C CNN
-F 3 "" H 14550 5550 50  0001 C CNN
-	1    14550 5550
-	1    0    0    -1
-$EndComp
-$Comp
 L power:GND #PWR?
 U 1 1 605141A5
@@
 	1    15100 6400
 	1    0    0    1
-$EndComp
-$Comp
-L power:+3.3V #PWR?
-U 1 1 6051520E
-P 15100 5550
-F 0 "#PWR?" H 15100 5400 50  0001 C CNN
-F 1 "+3.3V" H 15115 5723 50  0000 C CNN
-F 2 "" H 15100 5550 50  0001 C CNN
-F 3 "" H 15100 5550 50  0001 C CNN
-	1    15100 5550
-	1    0    0    -1
 $EndComp
 $Comp
@@
 NoConn ~ 4050 2350
 NoConn ~ 4050 2450
+$Comp
+L power:+1V8 #PWR?
+U 1 1 6010DD84
+P 9100 5550
+F 0 "#PWR?" H 9100 5400 50  0001 C CNN
+F 1 "+1V8" H 9115 5723 50  0000 C CNN
+F 2 "" H 9100 5550 50  0001 C CNN
+F 3 "" H 9100 5550 50  0001 C CNN
+	1    9100 5550
+	1    0    0    -1
+$EndComp
+$Comp
+L power:+1V8 #PWR?
+U 1 1 601158E8
+P 9700 5550
+F 0 "#PWR?" H 9700 5400 50  0001 C CNN
+F 1 "+1V8" H 9715 5723 50  0000 C CNN
+F 2 "" H 9700 5550 50  0001 C CNN
+F 3 "" H 9700 5550 50  0001 C CNN
+	1    9700 5550
+	1    0    0    -1
+$EndComp
+$Comp
+L power:+1V8 #PWR?
+U 1 1 60119540
+P 10250 5550
+F 0 "#PWR?" H 10250 5400 50  0001 C CNN
+F 1 "+1V8" H 10265 5723 50  0000 C CNN
+F 2 "" H 10250 5550 50  0001 C CNN
+F 3 "" H 10250 5550 50  0001 C CNN
+	1    10250 5550
+	1    0    0    -1
+$EndComp
+$Comp
+L power:+1V8 #PWR?
+U 1 1 6011D120
+P 10800 5550
+F 0 "#PWR?" H 10800 5400 50  0001 C CNN
+F 1 "+1V8" H 10815 5723 50  0000 C CNN
+F 2 "" H 10800 5550 50  0001 C CNN
+F 3 "" H 10800 5550 50  0001 C CNN
+	1    10800 5550
+	1    0    0    -1
+$EndComp
+$Comp
+L power:+1V8 #PWR?
+U 1 1 60120C1C
+P 11350 5550
+F 0 "#PWR?" H 11350 5400 50  0001 C CNN
+F 1 "+1V8" H 11365 5723 50  0000 C CNN
+F 2 "" H 11350 5550 50  0001 C CNN
+F 3 "" H 11350 5550 50  0001 C CNN
+	1    11350 5550
+	1    0    0    -1
+$EndComp
+$Comp
+L power:+1V8 #PWR?
+U 1 1 6012825E
+P 12900 5550
+F 0 "#PWR?" H 12900 5400 50  0001 C CNN
+F 1 "+1V8" H 12915 5723 50  0000 C CNN
+F 2 "" H 12900 5550 50  0001 C CNN
+F 3 "" H 12900 5550 50  0001 C CNN
+	1    12900 5550
+	1    0    0    -1
+$EndComp
+$Comp
+L power:+1V8 #PWR?
+U 1 1 6012BDD3
+P 13450 5550
+F 0 "#PWR?" H 13450 5400 50  0001 C CNN
+F 1 "+1V8" H 13465 5723 50  0000 C CNN
+F 2 "" H 13450 5550 50  0001 C CNN
+F 3 "" H 13450 5550 50  0001 C CNN
+	1    13450 5550
+	1    0    0    -1
+$EndComp
+$Comp
+L power:+1V8 #PWR?
+U 1 1 6012F9EB
+P 14000 5550
+F 0 "#PWR?" H 14000 5400 50  0001 C CNN
+F 1 "+1V8" H 14015 5723 50  0000 C CNN
+F 2 "" H 14000 5550 50  0001 C CNN
+F 3 "" H 14000 5550 50  0001 C CNN
+	1    14000 5550
+	1    0    0    -1
+$EndComp
+$Comp
+L power:+1V8 #PWR?
+U 1 1 601334E8
+P 14550 5550
+F 0 "#PWR?" H 14550 5400 50  0001 C CNN
+F 1 "+1V8" H 14565 5723 50  0000 C CNN
+F 2 "" H 14550 5550 50  0001 C CNN
+F 3 "" H 14550 5550 50  0001 C CNN
+	1    14550 5550
+	1    0    0    -1
+$EndComp
+$Comp
+L power:+1V8 #PWR?
+U 1 1 601370F7
+P 15100 5550
+F 0 "#PWR?" H 15100 5400 50  0001 C CNN
+F 1 "+1V8" H 15115 5723 50  0000 C CNN
+F 2 "" H 15100 5550 50  0001 C CNN
+F 3 "" H 15100 5550 50  0001 C CNN
+	1    15100 5550
+	1    0    0    -1
+$EndComp
 $EndSCHEMATC

Commit message: upd
Parts:
- gave numbers to parts that had none: 45
