File: Zynq-eame_UltraScale_0/KiCad/SUPPLY.sch (KiCad schematic (older format))
At the start: 1 part, among them U1 XCZU2CG

Commit message: UPD
Parts:
- added C? (x12): 10uF, Capacitor_SMD:C_0805_2012Metric, symbol Device:C
- added C? (x4): 100nF, Capacitor_SMD:C_0805_2012Metric, symbol Device:C
- added D?: LED_ALT, symbol Device:LED_ALT
- added J?: Barrel_Jack, symbol Connector:Barrel_Jack
- added L? (x4): 4.7uH, Inductor_SMD:L_Bourns-SRN1060, symbol Device:L
- added Q? (x4): MMBT3904, Package_TO_SOT_SMD:SOT-23, symbol Transistor_BJT:MMBT3904
- added R? (x3): 10k, Resistor_SMD:R_0805_2012Metric, symbol Device:R
- added R? (x2): 33k, Resistor_SMD:R_0805_2012Metric, symbol Device:R
- added R? (x4): 100k, Resistor_SMD:R_0805_2012Metric, symbol Device:R
- added R?: 75k, Resistor_SMD:R_0805_2012Metric, symbol Device:R
- added R? (x5): R, symbol Device:R
- added R?: 56k, Resistor_SMD:R_0805_2012Metric, symbol Device:R
- added SW?: SW_SPST, symbol Switch:SW_SPST
- added U? (x4): TPS563201, ZYNQ_7000:TPS563201, symbol Zynq_7000:TPS563201
Connections:
- net +1V8: now reaches U1.A21 (PS_MGTRAVTT)
- net +1V8: now also U1.AA5 (VCCO_PSIO0_500), U1.B19 (PS_MGTRAVTT), U1.B3 (VCCO_26), U1.B8 (VCCO_26), U1.C11 (VCCO_PSIO1_501), U1.C16 (VCCO_PSIO2_502), U1.C4 (VREF_66), U1.D14 (VCCO_PSIO2_502), U1.D19 (PS_MGTRAVTT), U1.E7 (VCCO_26), U1.F10 (VCCO_PSIO1_501), U1.G13 (VCCO_PSIO3_503), U1.G3 (VCCO_26), U1.H16 (VCCO_PSIO3_503), U1.J6 (VCCAUX_IO), U1.K2 (VCCO_26), U1.K5 (VREF_65), U1.K6 (VCCAUX_IO), U1.L13 (VCC_PSPLL), U1.L14 (VCC_PSPLL), U1.L16 (VCC_PSAUX), U1.L17 (VCC_PSAUX), U1.L6 (VCCAUX_IO), U1.M12 (VCC_PSPLL), U1.M16 (VCC_PSAUX), U1.M17 (VCC_PSAUX), U1.M20 (PS_MGTRREF_505), U1.M6 (VCCAUX), U1.P4 (VCCO_26), U1.P6 (VCCAUX), U1.V6 (VCCO_PSIO0_500), C?.2, C?.2, L?.2, R?.1, R?.1
- net +1V2: now reaches U1.AB18 (VCCO_PSDDR_504)
- net +1V2: now also U1.M14 (VCC_PSDDR_PLL), U1.M15 (VCC_PSDDR_PLL), U1.P19 (VCCO_PSDDR_504), U1.T20 (VCCO_PSDDR_504), U1.V16 (VCCO_PSDDR_504), U1.V21 (VCCO_PSDDR_504), U1.Y17 (VCCO_PSDDR_504), U1.Y22 (VCCO_PSDDR_504), C?.1, C?.1, L?.2, R?.2, R?.2
- net +1V0: now reaches U1.F19 (PS_MGTRAVCC)
- net +1V0: now also U1.H10 (VCCINT), U1.H19 (PS_MGTRAVCC), U1.H7 (VCCINT_IO), U1.H8 (VCCINT), U1.J11 (VCCINT), U1.J7 (VCCINT_IO), U1.J9 (VCCINT), U1.K19 (PS_MGTRAVCC), U1.K8 (VCCINT), U1.L11 (VCCINT), U1.L7 (VCCINT_IO), U1.M7 (VCCINT_IO), U1.M8 (VCCINT), U1.N11 (VCCINT), U1.N12 (VCC_PSINTLP), U1.N13 (VCC_PSINTLP), U1.N14 (VCC_PSINTFP), U1.N17 (VCC_PSINTFP_DDR), U1.N7 (VCCBRAM), U1.P10 (VCCINT), U1.P12 (VCC_PSINTLP), U1.P13 (VCC_PSINTLP), U1.P17 (VCC_PSINTFP_DDR), U1.P8 (VCCINT), U1.R11 (VCCINT), U1.R13 (VCC_PSINTLP), U1.R14 (VCC_PSINTLP), U1.R15 (VCC_PSINTFP), U1.R16 (VCC_PSINTFP), U1.R6 (VCCBRAM), U1.R7 (VCCBRAM), U1.R9 (VCCINT), U1.T12 (VCC_PSINTFP), U1.T13 (VCC_PSINTFP), U1.T14 (VCC_PSINTFP), U1.T16 (VCC_PSINTFP), U1.T17 (VCC_PSINTFP_DDR), U1.T6 (VCCBRAM), C?.1, C?.1, L?.2, Q?.1 (B), R?.1
- net GND: now reaches U1.N15 (VCC_PSBATT)
- net GND: now also C?.1, C?.1, C?.1, C?.2, C?.2, C?.2, C?.2, C?.2, C?.2, C?.2, C?.2, C?.2, D?.1 (K), J?.2, Q?.2 (E), Q?.2 (E), Q?.2 (E), Q?.2 (E), R?.1, R?.2, R?.2, R?.2, U?.1 (GND), U?.1 (GND), U?.1 (GND), U?.1 (GND)
- new net: C?.2, L?.1, U?.2 (SW)
- new net: R?.1, R?.2, U?.4 (VFB) (x4)
- new net: R?.1, U?.5 (EN)
- new net: C?.1, U?.6 (VBST)
- new net: C?.1, L?.1, U?.2 (SW) (x3)
- new net: Q?.3 (C), R?.2, U?.5 (EN)
- new net: C?.2, U?.6 (VBST) (x3)
- new net: R?.2, U?.5 (EN)
- new net: Q?.3 (C), R?.1, U?.5 (EN)
- new net: Q?.1 (B), Q?.3 (C), R?.2
- new net: Q?.1 (B), Q?.3 (C), R?.1
- new net: Q?.1 (B), R?.1
- new net: D?.2 (A), R?.1
- new net +3V3: C?.1, C?.1, L?.2, R?.1, R?.2
- new net +5V: J?.1, SW?.1 (A)
- new net VIN: C?.1, C?.1, C?.1, C?.2, R?.1, R?.1, R?.2, R?.2, R?.2, SW?.2 (B), U?.3 (IN), U?.3 (IN), U?.3 (IN), U?.3 (IN)
Other:
- note added: "LED ON"
- note added: "SUPPLY"
- note added: "VIN -> 1V0, 1V8, 1V2, 3V3"
- note added: "XCZU2CG"
- moved on the sheet: U1L

Commit message: upd
Parts:
- added +0V85?, +0V? (x8): +0V85, symbol Zynq_UltraScale:+0V85
- R?: value 33k -> 20K
- R?: value R -> 0R; footprint (none) -> Resistor_SMD:R_0805_2012Metric
- R? (x3): value R -> 10K; footprint (none) -> Resistor_SMD:R_0805_2012Metric
Connections:
- net +1V0 renamed +0V85
- net +0V85: now also +0V85?.~ (+0V85), +0V?.~ (+0V85), +0V?.~ (+0V85), +0V?.~ (+0V85), +0V?.~ (+0V85), +0V?.~ (+0V85), +0V?.~ (+0V85), +0V?.~ (+0V85), +0V?.~ (+0V85)
Other:
- note added: "VIN -> 0V85, 1V8, 1V2, 3V3"
- note removed: "VIN -> 1V0, 1V8, 1V2, 3V3"
Changed lines of the file:
@@
 Wire Wire Line
 	12750 5950 12800 5950
-$Comp
-L power:+1V0 #PWR?
-U 1 1 6061041D
-P 12550 5500
-F 0 "#PWR?" H 12550 5350 50  0001 C CNN
-F 1 "+1V0" V 12565 5628 50  0000 L CNN
-F 2 "" H 12550 5500 50  0001 C CNN
-F 3 "" H 12550 5500 50  0001 C CNN
-	1    12550 5500
-	0    -1   -1   0
-$EndComp
-Wire Wire Line
-	12550 5500 12750 5500
 Wire Wire Line
 	12750 5200 12800 5200
@@
 Wire Wire Line
 	12750 5400 12750 5500
-$Comp
-L power:+1V0 #PWR?
-U 1 1 6061F81B
-P 12550 7450
-F 0 "#PWR?" H 12550 7300 50  0001 C CNN
-F 1 "+1V0" V 12565 7578 50  0000 L CNN
-F 2 "" H 12550 7450 50  0001 C CNN
-F 3 "" H 12550 7450 50  0001 C CNN
-	1    12550 7450
-	0    -1   -1   0
-$EndComp
-Wire Wire Line
-	12550 7450 12750 7450
 Wire Wire Line
 	12800 7650 12750 7650
@@
 Wire Wire Line
 	12750 7750 12750 7850
-$Comp
-L power:+1V0 #PWR?
-U 1 1 60634A33
-P 12550 4950
-F 0 "#PWR?" H 12550 4800 50  0001 C CNN
-F 1 "+1V0" V 12565 5078 50  0000 L CNN
-F 2 "" H 12550 4950 50  0001 C CNN
-F 3 "" H 12550 4950 50  0001 C CNN
-	1    12550 4950
-	0    -1   -1   0
-$EndComp
-Wire Wire Line
-	12550 4950 12750 4950
 Wire Wire Line
 	12800 5050 12750 5050
@@
 	12800 4250 12750 4250
 Wire Wire Line
-	12750 4350 12750 4450
+	12750 4350 12750 4400
 Wire Wire Line
 	12750 4250 12750 4150
 Connection ~ 12750 4250
-$Comp
-L power:+1V0 #PWR?
-U 1 1 606540AA
-P 12550 4350
-F 0 "#PWR?" H 12550 4200 50  0001 C CNN
-F 1 "+1V0" V 12565 4478 50  0000 L CNN
-F 2 "" H 12550 4350 50  0001 C CNN
-F 3 "" H 12550 4350 50  0001 C CNN
-	1    12550 4350
-	0    -1   -1   0
-$EndComp
-Wire Wire Line
-	12550 4350 12750 4350
-$Comp
-L power:+1V0 #PWR?
-U 1 1 606592F0
-P 15000 6050
-F 0 "#PWR?" H 15000 5900 50  0001 C CNN
-F 1 "+1V0" V 15015 6178 50  0000 L CNN
-F 2 "" H 15000 6050 50  0001 C CNN
-F 3 "" H 15000 6050 50  0001 C CNN
-	1    15000 6050
-	0    1    1    0
-$EndComp
 Wire Wire Line
 	15000 6050 14800 6050
@@
 Wire Wire Line
 	14800 5950 14800 6050
-$Comp
-L power:+1V0 #PWR?
-U 1 1 6067C741
-P 15000 8050
-F 0 "#PWR?" H 15000 7900 50  0001 C CNN
-F 1 "+1V0" V 15015 8178 50  0000 L CNN
-F 2 "" H 15000 8050 50  0001 C CNN
-F 3 "" H 15000 8050 50  0001 C CNN
-	1    15000 8050
-	0    1    1    0
-$EndComp
 Wire Wire Line
 	15000 8050 14800 8050
@@
 Wire Wire Line
 	14800 8050 14800 8100
-$Comp
-L power:+1V0 #PWR?
-U 1 1 60690616
-P 15000 7500
-F 0 "#PWR?" H 15000 7350 50  0001 C CNN
-F 1 "+1V0" V 15015 7628 50  0000 L CNN
-F 2 "" H 15000 7500 50  0001 C CNN
-F 3 "" H 15000 7500 50  0001 C CNN
-	1    15000 7500
-	0    1    1    0
-$EndComp
 Wire Wire Line
 	15000 7500 14800 7500
@@
 P 4600 2100
 F 0 "R?" H 4670 2146 50  0000 L CNN
-F 1 "33k" H 4670 2055 50  0000 L CNN
+F 1 "20K" H 4670 2055 50  0000 L CNN
 F 2 "Resistor_SMD:R_0805_2012Metric" V 4530 2100 50  0001 C CNN
 F 3 "~" H 4600 2100 50  0001 C CNN
@@
 P 2600 6250
 F 0 "R?" V 2393 6250 50  0000 C CNN
-F 1 "R" V 2484 6250 50  0000 C CNN
-F 2 "" V 2530 6250 50  0001 C CNN
+F 1 "0R" V 2484 6250 50  0000 C CNN
+F 2 "Resistor_SMD:R_0805_2012Metric" V 2530 6250 50  0001 C CNN
 F 3 "~" H 2600 6250 50  0001 C CNN
 	1    2600 6250
@@
 P 2650 8250
 F 0 "R?" V 2443 8250 50  0000 C CNN
-F 1 "R" V 2534 8250 50  0000 C CNN
-F 2 "" V 2580 8250 50  0001 C CNN
+F 1 "10K" V 2534 8250 50  0000 C CNN
+F 2 "Resistor_SMD:R_0805_2012Metric" V 2580 8250 50  0001 C CNN
 F 3 "~" H 2650 8250 50  0001 C CNN
 	1    2650 8250
@@
 P 2150 8250
 F 0 "R?" V 1943 8250 50  0000 C CNN
-F 1 "R" V 2034 8250 50  0000 C CNN
-F 2 "" V 2080 8250 50  0001 C CNN
+F 1 "10K" V 2034 8250 50  0000 C CNN
+F 2 "Resistor_SMD:R_0805_2012Metric" V 2080 8250 50  0001 C CNN
 F 3 "~" H 2150 8250 50  0001 C CNN
 	1    2150 8250
@@
 P 1600 9000
 F 0 "R?" V 1393 9000 50  0000 C CNN
-F 1 "R" V 1484 9000 50  0000 C CNN
-F 2 "" V 1530 9000 50  0001 C CNN
+F 1 "10K" V 1484 9000 50  0000 C CNN
+F 2 "Resistor_SMD:R_0805_2012Metric" V 1530 9000 50  0001 C CNN
 F 3 "~" H 1600 9000 50  0001 C CNN
 	1    1600 9000
@@
 Wire Wire Line
 	2650 8450 2650 8400
-$Comp
-L power:+1V0 #PWR?
-U 1 1 615A0715
-P 5200 1800
-F 0 "#PWR?" H 5200 1650 50  0001 C CNN
-F 1 "+1V0" H 5215 1973 50  0000 C CNN
-F 2 "" H 5200 1800 50  0001 C CNN
-F 3 "" H 5200 1800 50  0001 C CNN
-	1    5200 1800
-	1    0    0    -1
-$EndComp
 Wire Wire Line
 	5200 1800 5200 1900
@@
 Wire Wire Line
 	1850 6450 1850 6550
-$Comp
-L power:+1V0 #PWR?
-U 1 1 61650CDA
-P 1750 4700
-F 0 "#PWR?" H 1750 4550 50  0001 C CNN
-F 1 "+1V0" H 1600 4750 50  0000 C CNN
-F 2 "" H 1750 4700 50  0001 C CNN
-F 3 "" H 1750 4700 50  0001 C CNN
-	1    1750 4700
-	1    0    0    -1
-$EndComp
 Wire Wire Line
 	1750 4700 1750 4750
@@
 LED ON
 Text Notes 4050 950  2    118  ~ 24
-VIN -> 1V0, 1V8, 1V2, 3V3
+VIN -> 0V85, 1V8, 1V2, 3V3
 Text Notes 11250 1050 2    118  ~ 24
 XCZU2CG
+Wire Wire Line
+	12500 4400 12750 4400
+Connection ~ 12750 4400
+Wire Wire Line
+	12750 4400 12750 4450
+$Comp
+L Zynq_UltraScale:+0V85 +0V85?
+U 1 1 6081C189
+P 12500 4400
+F 0 "+0V85?" H 12500 4350 50  0001 C CNN
+F 1 "+0V85" V 12500 4550 50  0000 L CNN
+F 2 "" H 12500 4350 50  0001 C CNN
+F 3 "" H 12500 4350 50  0001 C CNN
+	1    12500 4400
+	0    -1   -1   0
+$EndComp
+$Comp
+L Zynq_UltraScale:+0V85 +0V?
+U 1 1 608A27EF
+P 12500 4950
+F 0 "+0V?" H 12500 4900 50  0001 C CNN
+F 1 "+0V85" V 12500 5100 50  0000 L CNN
+F 2 "" H 12500 4900 50  0001 C CNN
+F 3 "" H 12500 4900 50  0001 C CNN
+	1    12500 4950
+	0    -1   -1   0
+$EndComp
+Wire Wire Line
+	12500 4950 12750 4950
+$Comp
+L Zynq_UltraScale:+0V85 +0V?
+U 1 1 609074CA
+P 12500 5500
+F 0 "+0V?" H 12500 5450 50  0001 C CNN
+F 1 "+0V85" V 12500 5650 50  0000 L CNN
+F 2 "" H 12500 5450 50  0001 C CNN
+F 3 "" H 12500 5450 50  0001 C CNN
+	1    12500 5500
+	0    -1   -1   0
+$EndComp
+Wire Wire Line
+	12500 5500 12750 5500
+$Comp
+L Zynq_UltraScale:+0V85 +0V?
+U 1 1 6096BF23
+P 12450 7450
+F 0 "+0V?" H 12450 7400 50  0001 C CNN
+F 1 "+0V85" V 12450 7600 50  0000 L CNN
+F 2 "" H 12450 7400 50  0001 C CNN
+F 3 "" H 12450 7400 50  0001 C CNN
+	1    12450 7450
+	0    -1   -1   0
+$EndComp
+Wire Wire Line
+	12450 7450 12750 7450
+$Comp
+L Zynq_UltraScale:+0V85 +0V?
+U 1 1 609F2065
+P 15000 8050
+F 0 "+0V?" H 15000 8000 50  0001 C CNN
+F 1 "+0V85" V 15000 8200 50  0000 L CNN
+F 2 "" H 15000 8000 50  0001 C CNN
+F 3 "" H 15000 8000 50  0001 C CNN
+	1    15000 8050
+	0    1    1    0
+$EndComp
+$Comp
+L Zynq_UltraScale:+0V85 +0V?
+U 1 1 60A1362E
+P 15000 7500
+F 0 "+0V?" H 15000 7450 50  0001 C CNN
+F 1 "+0V85" V 15000 7650 50  0000 L CNN
+F 2 "" H 15000 7450 50  0001 C CNN
+F 3 "" H 15000 7450 50  0001 C CNN
+	1    15000 7500
+	0    1    1    0
+$EndComp
+$Comp
+L Zynq_UltraScale:+0V85 +0V?
+U 1 1 60A34B10
+P 15000 6050
+F 0 "+0V?" H 15000 6000 50  0001 C CNN
+F 1 "+0V85" V 15000 6200 50  0000 L CNN
+F 2 "" H 15000 6000 50  0001 C CNN
+F 3 "" H 15000 6000 50  0001 C CNN
+	1    15000 6050
+	0    1    1    0
+$EndComp
+$Comp
+L Zynq_UltraScale:+0V85 +0V?
+U 1 1 60A774B0
+P 5200 1800
+F 0 "+0V?" H 5200 1750 50  0001 C CNN
+F 1 "+0V85" H 5050 1950 50  0000 L CNN
+F 2 "" H 5200 1750 50  0001 C CNN
+F 3 "" H 5200 1750 50  0001 C CNN
+	1    5200 1800
+	1    0    0    -1
+$EndComp
+$Comp
+L Zynq_UltraScale:+0V85 +0V?
+U 1 1 60AC23C2
+P 1750 4700
+F 0 "+0V?" H 1750 4650 50  0001 C CNN
+F 1 "+0V85" H 1450 4750 50  0000 L CNN
+F 2 "" H 1750 4650 50  0001 C CNN
+F 3 "" H 1750 4650 50  0001 C CNN
+	1    1750 4700
+	1    0    0    -1
+$EndComp
 $EndSCHEMATC

Commit message: upd
Parts:
- removed +0V85?, +0V? (x8): +0V85, symbol Zynq_UltraScale:+0V85
- gave numbers to parts that had none: 47
