File: Zynq-eame_UltraScale_0/KiCad/Zynq-eame_UltraScale_0.kicad_pcb (KiCad board)
At the start: 2 copper layers, 33 parts, among them J1 USB_B_Micro, J2 Conn_01x06, SW1 SW_Push, U1 XCZU2CG, U2 MT40A512M16, U3 FT2232H, U4 93C46, Y1 12MHz

Commit message: UPD
Parts:
- added C15: 100nF, Capacitor_SMD:C_0805_2012Metric, F.Cu at (136.9, 100.1)
- added C16: 100nF, Capacitor_SMD:C_0805_2012Metric, F.Cu at (143.9, 87.6)
- added C17: 100nF, Capacitor_SMD:C_0805_2012Metric, F.Cu at (139.4, 93.6)
- added C18: 100nF, Capacitor_SMD:C_0805_2012Metric, F.Cu at (136.9, 97.1)
- added D2: LED_ALT, LED_SMD:LED_0805_2012Metric, F.Cu at (139.4, 87.6)
- added R12: 1K, Resistor_SMD:R_0805_2012Metric, F.Cu at (148.3, 87.6)
- added R13: 1K, Resistor_SMD:R_0805_2012Metric, F.Cu at (143.8, 93.5)
- added R14: 820, Resistor_SMD:R_0805_2012Metric, F.Cu at (139.4, 90.6)
- added R15: 1300, Resistor_SMD:R_0805_2012Metric, F.Cu at (141.3, 96.5)
- added R16: 4.7K, Resistor_SMD:R_0805_2012Metric, F.Cu at (148.3, 90.5)
- added R17: 10k, Resistor_SMD:R_0805_2012Metric, F.Cu at (152.7, 87.6)
- added R18: 330, Resistor_SMD:R_0805_2012Metric, F.Cu at (148.2, 93.5)
- added R19: 4.7K, Resistor_SMD:R_0805_2012Metric, F.Cu at (141.3, 99.5)
- added R9: 10k, Resistor_SMD:R_0805_2012Metric, F.Cu at (143.9, 90.5)
- added U6: IP4856CX25, Zynq-eame_UltraScale_0:BGA-25_5x5_2.049999x2.049999mm, F.Cu at (145.3, 96.7)
- added U7: MT25QU512ABB, Zynq-eame_UltraScale_0:BGA-25_5x5_6.0x8.0mm, F.Cu at (133.4, 90.9)
- added X1: ASE-33.333MHz, Oscillator:Oscillator_SMD_Abracon_ASE-4Pin_3.2x2.5mm, F.Cu at (132.2, 97.9)
Connections:
- U1 pad A12: (no net) -> /MIO&REFERENCE/MIO_SD1_DAT3
- U1 pad A13: (no net) -> /MIO&REFERENCE/MIO_SD1_CMD
- U1 pad AA1: (no net) -> /MIO&REFERENCE/QSPI_CS
- U1 pad B10: (no net) -> /MIO&REFERENCE/MIO_SD1_DIR_DAT0
- U1 pad B12: (no net) -> /MIO&REFERENCE/MIO_SD1_DAT1
- U1 pad C12: (no net) -> /MIO&REFERENCE/MIO_SD1_DAT0
- U1 pad C13: (no net) -> /MIO&REFERENCE/MIO_SD1_CLK
- U1 pad D11: (no net) -> /MIO&REFERENCE/MIO_SD1_DIR_CMD
- U1 pad D13: (no net) -> /MIO&REFERENCE/MIO_SD1_DAT2
- U1 pad H14: (no net) -> /MIO&REFERENCE/PS_CLK
- U1 pad H17: (no net) -> GND
- U1 pad K12: (no net) -> /MIO&REFERENCE/PS_POR_B
- U1 pad K16: (no net) -> /MIO&REFERENCE/PS_ERROR
- U1 pad U4: (no net) -> /MIO&REFERENCE/QSPI_CLK
- U1 pad U5: (no net) -> /MIO&REFERENCE/QSPI_DQ3
- U1 pad U6: (no net) -> /MIO&REFERENCE/QSPI_DQ0
- U1 pad V2: (no net) -> /MIO&REFERENCE/QSPI_DQ2
- U1 pad W1: (no net) -> /MIO&REFERENCE/QSPI_DQ1

Commit message: upd
Parts:
- added C19: 10uF, Capacitor_SMD:C_0805_2012Metric, F.Cu at (163.8, 52.2)
- added C20: 10uF, Capacitor_SMD:C_0805_2012Metric, F.Cu at (163.8, 55.1)
- added C21: 10uF, Capacitor_SMD:C_0805_2012Metric, F.Cu at (165.0, 49.2)
- added C22: 10uF, Capacitor_SMD:C_0805_2012Metric, F.Cu at (153.9, 61.1)
- added C23: 100nF, Capacitor_SMD:C_0805_2012Metric, F.Cu at (159.4, 53.7)
- added C24: 100nF, Capacitor_SMD:C_0805_2012Metric, F.Cu at (137.7, 61.0)
- added C25: 100nF, Capacitor_SMD:C_0805_2012Metric, F.Cu at (177.3, 46.1)
- added C26: 100nF, Capacitor_SMD:C_0805_2012Metric, F.Cu at (133.3, 61.0)
- added C27: 10uF, Capacitor_SMD:C_0805_2012Metric, F.Cu at (160.6, 49.1)
- added C28: 10uF, Capacitor_SMD:C_0805_2012Metric, F.Cu at (155.0, 53.7)
- added C29: 10uF, Capacitor_SMD:C_0805_2012Metric, F.Cu at (149.5, 58.1)
- added C30: 10uF, Capacitor_SMD:C_0805_2012Metric, F.Cu at (174.1, 37.3)
- added C31: 10uF, Capacitor_SMD:C_0805_2012Metric, F.Cu at (149.5, 61.1)
- added C32: 10uF, Capacitor_SMD:C_0805_2012Metric, F.Cu at (168.5, 46.3)
- added C33: 10uF, Capacitor_SMD:C_0805_2012Metric, F.Cu at (174.1, 40.2)
- added C34: 10uF, Capacitor_SMD:C_0805_2012Metric, F.Cu at (153.9, 58.1)
- added C35: 4.7uF, Capacitor_SMD:C_0805_2012Metric, F.Cu at (140.5, 71.1)
- added C36: 100nF, Capacitor_SMD:C_0805_2012Metric, F.Cu at (140.5, 68.1)
- added C37: 100nF, Capacitor_SMD:C_0805_2012Metric, F.Cu at (185.8, 65.6)
- added L3: 4.7uH, Inductor_SMD:L_Bourns-SRN1060, F.Cu at (219.3, 82.1)
- added L4: 4.7uH, Inductor_SMD:L_Bourns-SRN1060, F.Cu at (207.8, 97.8)
- added L5: 4.7uH, Inductor_SMD:L_Bourns-SRN1060, F.Cu at (207.6, 82.1)
- added L6: 4.7uH, Inductor_SMD:L_Bourns-SRN1060, F.Cu at (231.0, 82.1)
- added Q1: MMBT3904, Package_TO_SOT_SMD:SOT-23, F.Cu at (156.2, 49.9)
- added Q2: MMBT3904, Package_TO_SOT_SMD:SOT-23, F.Cu at (150.6, 54.4)
- added Q3: MMBT3904, Package_TO_SOT_SMD:SOT-23, F.Cu at (145.0, 58.8)
- added Q4: MMBT3904, Package_TO_SOT_SMD:SOT-23, F.Cu at (168.5, 42.5)
- added Q5: MMBF170, Package_TO_SOT_SMD:SOT-23, F.Cu at (206.7, 42.6)
- added Q6: MMBF170, Package_TO_SOT_SMD:SOT-23, F.Cu at (190.2, 55.6)
- added Q7: MMBF170, Package_TO_SOT_SMD:SOT-23, F.Cu at (206.7, 38.1)
- added Q8: MMBF170, Package_TO_SOT_SMD:SOT-23, F.Cu at (185.8, 55.6)
- added Q9: MMBF170, Package_TO_SOT_SMD:SOT-23, F.Cu at (196.2, 49.8)
- added R20: 10K, Resistor_SMD:R_0805_2012Metric, F.Cu at (172.7, 55.1)
- added R21: 10K, Resistor_SMD:R_0805_2012Metric, F.Cu at (167.1, 58.1)
- added R22: 10k, Resistor_SMD:R_0805_2012Metric, F.Cu at (172.7, 52.2)
- added R23: 10k, Resistor_SMD:R_0805_2012Metric, F.Cu at (173.8, 49.2)
- added R24: 10k, Resistor_SMD:R_0805_2012Metric, F.Cu at (178.2, 49.1)
- added R25: 0R, Resistor_SMD:R_0805_2012Metric, F.Cu at (172.9, 43.2)
- added R26: 10K, Resistor_SMD:R_0805_2012Metric, F.Cu at (172.9, 46.3)
- added R27: 100k, Resistor_SMD:R_0805_2012Metric, F.Cu at (158.3, 59.6)
- added R28: 75k, Resistor_SMD:R_0805_2012Metric, F.Cu at (162.7, 61.0)
- added R29: 56k, Resistor_SMD:R_0805_2012Metric, F.Cu at (169.4, 49.2)
- added R30: 100k, Resistor_SMD:R_0805_2012Metric, F.Cu at (168.3, 52.2)
- added R31: 33k, Resistor_SMD:R_0805_2012Metric, F.Cu at (177.4, 43.2)
- added R32: 100k, Resistor_SMD:R_0805_2012Metric, F.Cu at (162.7, 58.1)
- added R33: 20K, Resistor_SMD:R_0805_2012Metric, F.Cu at (158.3, 56.6)
- added R34: 100k, Resistor_SMD:R_0805_2012Metric, F.Cu at (168.3, 55.1)
- added R36: 1K, Resistor_SMD:R_0805_2012Metric, F.Cu at (205.1, 52.3)
- added R37: 4.7K, Resistor_SMD:R_0805_2012Metric, F.Cu at (211.1, 37.3)
- added R38: 10K, Resistor_SMD:R_0805_2012Metric, F.Cu at (200.7, 49.0)
- added R39: 4.7K, Resistor_SMD:R_0805_2012Metric, F.Cu at (206.7, 46.4)
- added R40: 4.7K, Resistor_SMD:R_0805_2012Metric, F.Cu at (215.5, 37.3)
- added R41: 4.7K, Resistor_SMD:R_0805_2012Metric, F.Cu at (211.1, 40.2)
- added R42: 1K, Resistor_SMD:R_0805_2012Metric, F.Cu at (200.7, 51.9)
- added R43: 10K, Resistor_SMD:R_0805_2012Metric, F.Cu at (205.1, 49.3)
- added R44: 4.7K, Resistor_SMD:R_0805_2012Metric, F.Cu at (199.1, 54.9)
- added R45: 4.7K, Resistor_SMD:R_0805_2012Metric, F.Cu at (207.9, 55.2)
- added R46: 4.7K, Resistor_SMD:R_0805_2012Metric, F.Cu at (215.5, 40.2)
- added R47: 1K, Resistor_SMD:R_0805_2012Metric, F.Cu at (211.1, 43.2)
- added R48: 10K, Resistor_SMD:R_0805_2012Metric, F.Cu at (211.1, 46.4)
- added R49: 4.7K, Resistor_SMD:R_0805_2012Metric, F.Cu at (194.7, 54.8)
- added R50: 4.7K, Resistor_SMD:R_0805_2012Metric, F.Cu at (213.9, 52.3)
- added R51: 1K, Resistor_SMD:R_0805_2012Metric, F.Cu at (219.9, 46.1)
- added R52: 4.7K, Resistor_SMD:R_0805_2012Metric, F.Cu at (219.9, 43.2)
- added R53: 10K, Resistor_SMD:R_0805_2012Metric, F.Cu at (213.9, 49.3)
- added R54: 4.7K, Resistor_SMD:R_0805_2012Metric, F.Cu at (209.5, 52.3)
- added R55: 4.7K, Resistor_SMD:R_0805_2012Metric, F.Cu at (215.5, 46.1)
- added R56: 4.7K, Resistor_SMD:R_0805_2012Metric, F.Cu at (203.5, 55.2)
- added R57: 1K, Resistor_SMD:R_0805_2012Metric, F.Cu at (219.9, 40.2)
- added R58: 4.7K, Resistor_SMD:R_0805_2012Metric, F.Cu at (215.5, 43.2)
- added R59: 10K, Resistor_SMD:R_0805_2012Metric, F.Cu at (209.5, 49.3)
- added R60: 4.7K, Resistor_SMD:R_0805_2012Metric, F.Cu at (219.9, 37.3)
- added R61: 4.7k, Resistor_SMD:R_0805_2012Metric, F.Cu at (144.9, 71.1)
- added R62: 10k, Resistor_SMD:R_0805_2012Metric, F.Cu at (140.5, 74.0)
- added R63: 1k, Resistor_SMD:R_0805_2012Metric, F.Cu at (144.9, 68.1)
- added R64: 300, Resistor_SMD:R_0805_2012Metric, F.Cu at (194.6, 62.6)
- added R65: 1K, Resistor_SMD:R_0805_2012Metric, F.Cu at (190.2, 65.6)
- added R66: 240, Resistor_SMD:R_0805_2012Metric, F.Cu at (190.2, 62.6)
- added R67: 240, Resistor_SMD:R_0805_2012Metric, F.Cu at (185.8, 62.6)
- added SW3: SW_SPST, Button_Switch_SMD:SW_DIP_SPSTx01_Slide_6.7x4.1mm_W6.73mm_P2.54mm_LowProfile_JPin, F.Cu at (188.8, 50.4)
- added SW4: SW_SPST, Button_Switch_SMD:SW_DIP_SPSTx01_Slide_6.7x4.1mm_W6.73mm_P2.54mm_LowProfile_JPin, F.Cu at (199.2, 44.6)
- added SW5: SW_SPST, Button_Switch_SMD:SW_DIP_SPSTx01_Slide_6.7x4.1mm_W6.73mm_P2.54mm_LowProfile_JPin, F.Cu at (188.8, 38.7)
- added SW6: SW_SPST, Button_Switch_SMD:SW_DIP_SPSTx01_Slide_6.7x4.1mm_W6.73mm_P2.54mm_LowProfile_JPin, F.Cu at (188.8, 44.6)
- added SW7: SW_SPST, Button_Switch_SMD:SW_DIP_SPSTx01_Slide_6.7x4.1mm_W6.73mm_P2.54mm_LowProfile_JPin, F.Cu at (199.2, 38.7)
- added U10: TPS563201, ZYNQ_7000:TPS563201, F.Cu at (145.7, 49.9)
- added U11: TPS563201, ZYNQ_7000:TPS563201, F.Cu at (151.2, 49.9)
- added U12: CP2102N-A01-GQFN28, Package_DFN_QFN:QFN-28-1EP_5x5mm_P0.5mm_EP3.35x3.35mm, F.Cu at (134.7, 70.3)
- added U8: TPS563201, ZYNQ_7000:TPS563201, F.Cu at (169.1, 38.0)
- added U9: TPS563201, ZYNQ_7000:TPS563201, F.Cu at (145.7, 54.3)
- moved R8 7.93 mm to (151.0, 43.9)
Connections:
- U1 pad A21: (no net) -> +1V8
- U1 pad AA13: (no net) -> /DDR/DDR_DQS_N1
- U1 pad AA5: (no net) -> +1V8
- U1 pad AA9: (no net) -> /DDR/DDR_DQS_N0
- U1 pad AB14: (no net) -> /DDR/DDR_DM1
- U1 pad AB18: (no net) -> +1V2
- U1 pad AB9: (no net) -> /DDR/DDR_DM0
- U1 pad B19: (no net) -> +1V8
- U1 pad B3: (no net) -> +1V8
- U1 pad B8: (no net) -> +1V8
- U1 pad C11: (no net) -> +1V8
- U1 pad C16: (no net) -> +1V8
- U1 pad C4: (no net) -> +1V8
- U1 pad D14: (no net) -> +1V8
- U1 pad D19: (no net) -> +1V8
- U1 pad E7: (no net) -> +1V8
- U1 pad F10: (no net) -> +1V8
- U1 pad F19: (no net) -> +0V85
- U1 pad F4: (no net) -> /PINOUT/BT_1
- U1 pad G13: (no net) -> +1V8
- U1 pad G2: (no net) -> /PINOUT/BT_5
- U1 pad G3: (no net) -> +1V8
- U1 pad G4: (no net) -> /PINOUT/BT_3
- U1 pad H10: (no net) -> +0V85
- U1 pad H16: (no net) -> +1V8
- U1 pad H19: (no net) -> +0V85
- U1 pad H2: (no net) -> /PINOUT/SW_1
- U1 pad H3: (no net) -> /PINOUT/BT_2
- U1 pad H4: (no net) -> /PINOUT/BT_4
- U1 pad H5: (no net) -> /PINOUT/SW_2
- U1 pad H7: (no net) -> +0V85
- U1 pad H8: (no net) -> +0V85
- U1 pad J1: (no net) -> /PINOUT/SW_4
- U1 pad J11: (no net) -> +0V85
- U1 pad J2: (no net) -> /PINOUT/LED_3
- U1 pad J3: (no net) -> /PINOUT/LED_4
- U1 pad J5: (no net) -> /PINOUT/SW_3
- U1 pad J6: (no net) -> +1V8
- U1 pad J7: (no net) -> +0V85
- U1 pad J9: (no net) -> +0V85
- U1 pad K1: (no net) -> /PINOUT/SW_5
- U1 pad K19: (no net) -> +0V85
- U1 pad K2: (no net) -> +1V8
- U1 pad K3: (no net) -> /PINOUT/LED_1
- U1 pad K4: (no net) -> /PINOUT/LED_2
- U1 pad K5: (no net) -> +1V8
- U1 pad K6: (no net) -> +1V8
- U1 pad K8: (no net) -> +0V85
- U1 pad L11: (no net) -> +0V85
- U1 pad L13: (no net) -> +1V8
- U1 pad L14: (no net) -> +1V8
- U1 pad L16: (no net) -> +1V8
- U1 pad L17: (no net) -> +1V8
- U1 pad L3: (no net) -> /PINOUT/LED_5
- U1 pad L6: (no net) -> +1V8
- U1 pad L7: (no net) -> +0V85
- U1 pad M12: (no net) -> +1V8
- U1 pad M14: (no net) -> +1V2
- U1 pad M15: (no net) -> +1V2
- U1 pad M16: (no net) -> +1V8
- U1 pad M17: (no net) -> +1V8
- U1 pad M20: (no net) -> +1V8
- U1 pad M6: (no net) -> +1V8
- U1 pad M7: (no net) -> +0V85
- U1 pad M8: (no net) -> +0V85
- U1 pad N11: (no net) -> +0V85
- U1 pad N12: (no net) -> +0V85
- U1 pad N13: (no net) -> +0V85
- U1 pad N14: (no net) -> +0V85
- U1 pad N15: (no net) -> GND
- U1 pad N17: (no net) -> +0V85
- U1 pad N7: (no net) -> +0V85
- U1 pad P10: (no net) -> +0V85
- U1 pad P12: (no net) -> +0V85
- U1 pad P13: (no net) -> +0V85
- U1 pad P17: (no net) -> +0V85
- U1 pad P19: (no net) -> +1V2
- U1 pad P4: (no net) -> +1V8
- U1 pad P6: (no net) -> +1V8
- U1 pad P8: (no net) -> +0V85
- U1 pad R11: (no net) -> +0V85
- U1 pad R13: (no net) -> +0V85
- U1 pad R14: (no net) -> +0V85
- U1 pad R15: (no net) -> +0V85
- U1 pad R16: (no net) -> +0V85
- U1 pad R6: (no net) -> +0V85
- U1 pad R7: (no net) -> +0V85
- U1 pad R9: (no net) -> +0V85
- U1 pad T12: (no net) -> +0V85
- U1 pad T13: (no net) -> +0V85
- U1 pad T14: (no net) -> +0V85
- U1 pad T16: (no net) -> +0V85
- U1 pad T17: (no net) -> +0V85
- U1 pad T19: (no net) -> Net-(R67-Pad1)
- U1 pad T20: (no net) -> +1V2
- U1 pad T6: (no net) -> +0V85
- U1 pad U16: (no net) -> /DDR/DDR_BG0
- U1 pad U17: (no net) -> /DDR/DDR_BA0
- U1 pad U22: (no net) -> /DDR/DDR_CKE
- U1 pad V16: (no net) -> +1V2
- U1 pad V17: (no net) -> /DDR/DDR_BA1
- U1 pad V20: (no net) -> /DDR/DDR_CK
- U1 pad V21: (no net) -> +1V2
- U1 pad V22: (no net) -> /DDR/DDR_CS
- U1 pad V3: (no net) -> /MIO&REFERENCE/MIO8_TX
- U1 pad V5: (no net) -> /MIO&REFERENCE/MIO9_RX
- U1 pad V6: (no net) -> +1V8
- U1 pad W20: (no net) -> /DDR/DDR_CK_N
- U1 pad W22: (no net) -> /DDR/DDR_ODT
- U1 pad Y13: (no net) -> /DDR/DDR_DQS_P1
- U1 pad Y17: (no net) -> +1V2
- U1 pad Y22: (no net) -> +1V2
- U1 pad Y9: (no net) -> /DDR/DDR_DQS_P0
- U2 pad A7: (no net) -> /DDR/DDR_DQS_N1
- U2 pad B1: (no net) -> +2V5
- U2 pad B7: (no net) -> /DDR/DDR_DQS_P1
- U2 pad E2: (no net) -> /DDR/DDR_DM1
- U2 pad E7: (no net) -> /DDR/DDR_DM0
- U2 pad F3: (no net) -> /DDR/DDR_DQS_N0
- U2 pad F9: (no net) -> Net-(R66-Pad1)
- U2 pad G3: (no net) -> /DDR/DDR_DQS_P0
- U2 pad K2: (no net) -> /DDR/DDR_CKE
- U2 pad K3: (no net) -> /DDR/DDR_ODT
- U2 pad K7: (no net) -> /DDR/DDR_CK
- U2 pad K8: (no net) -> /DDR/DDR_CK_N
- U2 pad L7: (no net) -> /DDR/DDR_CS
- U2 pad M1: (no net) -> Net-(C37-Pad2)
- U2 pad M2: (no net) -> /DDR/DDR_BG0
- U2 pad N2: (no net) -> /DDR/DDR_BA0
- U2 pad N8: (no net) -> /DDR/DDR_BA1
- U2 pad N9: (no net) -> GND
- U2 pad R9: (no net) -> +2V5
