File: Zynq-eame_UltraScale_0/KiCad/DDR.sch (KiCad schematic (older format))
At the start: 35 parts, among them U5 XC7Z010-BUENO, U6 MT41K256M16TW-107_P, U7 MT41K256M16TW-107_P

Commit message: update
Parts:
- removed C17, C18, C19, C20, C21, C22, C23, C24, C25, C26, C27, C28, C29, C30, C31, C32, C33, C34, C53, C54, C55, C56, C57, C58, C59, C60: 100nF, Capacitor_SMD:C_0805_2012Metric, symbol Device:C
- removed R18, R23: 240R 1%, Resistor_SMD:R_0805_2012Metric, symbol Device:R
- removed R19, R20, R21, R22: 1k 1%, Resistor_SMD:R_0805_2012Metric, symbol Device:R
- removed U5: XC7Z010-BUENO, ZYNQ_7000:BGA-400_20x20_17.0x17.0mm, symbol Zynq_7000:XC7Z010-BUENO
- removed U6, U7: MT41K256M16TW-107_P, ZYNQ_7000:BGA-144_9x16_8.0x14.0mm, symbol Zynq_7000:MT41K256M16TW-107_P
- added U1: XCZU2CG, Zynq-eame_UltraScale_0:SBVA484, symbol Zynq_UltraScale:XCZU2CG
- added U2: MT40A512M16, Zynq-eame_UltraScale_0:FBGA96_LY, symbol Zynq_UltraScale:MT40A512M16
Connections:
- net DDR_A0: now also U1.AA22 (PS_DDR_A0), U2.P3 (A0)
- net DDR_A1: now also U1.AB20 (PS_DDR_A1), U2.P7 (A1)
- net DDR_A10: now also U1.Y21 (PS_DDR_A10), U2.M3 (A10/AP)
- net DDR_A11: now also U1.AA21 (PS_DDR_A11), U2.T2 (A11)
- net DDR_A12: now also U1.AA18 (PS_DDR_A12), U2.M7 (A12/BC_n)
- net DDR_A13: now also U1.AA19 (PS_DDR_A13), U2.T8 (A13)
- net DDR_A14: now also U1.AA17 (PS_DDR_A14), U2.L2 (WE_n/A14)
- net DDR_A2: now also U1.AB17 (PS_DDR_A2), U2.R3 (A2)
- net DDR_A3: now also U1.AB19 (PS_DDR_A3), U2.N7 (A3)
- net DDR_A4: now also U1.AB21 (PS_DDR_A4), U2.N3 (A4)
- net DDR_A5: now also U1.AB16 (PS_DDR_A5), U2.P8 (A5)
- net DDR_A6: now also U1.Y20 (PS_DDR_A6), U2.P2 (A6)
- net DDR_A7: now also U1.Y19 (PS_DDR_A7), U2.R8 (A7)
- net DDR_A8: now also U1.W17 (PS_DDR_A8), U2.R2 (A8)
- net DDR_A9: now also U1.Y18 (PS_DDR_A9), U2.R7 (A9)
- net DDR_D0: now also U1.AB11 (PS_DDR_DQ0), U2.G2 (DQ0)
- net DDR_D1: now also U1.Y10 (PS_DDR_DQ1), U2.F7 (DQ1)
- net DDR_D10: now also U1.AA12 (PS_DDR_DQ10), U2.C3 (DQ10)
- net DDR_D11: now also U1.AB12 (PS_DDR_DQ11), U2.C7 (DQ11)
- net DDR_D12: now also U1.Y14 (PS_DDR_DQ12), U2.C2 (DQ12)
- net DDR_D13: now also U1.AA14 (PS_DDR_DQ13), U2.C8 (DQ13)
- net DDR_D14: now also U1.Y15 (PS_DDR_DQ14), U2.D3 (DQ14)
- net DDR_D15: now also U1.AB15 (PS_DDR_DQ15), U2.D7 (DQ15)
- net DDR_D2: now also U1.AB10 (PS_DDR_DQ2), U2.H3 (DQ2)
- net DDR_D3: now also U1.W10 (PS_DDR_DQ3), U2.H7 (DQ3)
- net DDR_D4: now also U1.AA8 (PS_DDR_DQ4), U2.H2 (DQ4)
- net DDR_D5: now also U1.Y8 (PS_DDR_DQ5), U2.H8 (DQ5)
- net DDR_D6: now also U1.AB7 (PS_DDR_DQ6), U2.J3 (DQ6)
- net DDR_D7: now also U1.AA7 (PS_DDR_DQ7), U2.J7 (DQ7)
- net DDR_D8: now also U1.AA11 (PS_DDR_DQ8), U2.A3 (DQ8)
- net DDR_D9: now also U1.Y11 (PS_DDR_DQ9), U2.B8 (DQ9)
- net DDR_RESETN: now also U1.T18 (PS_DDR_RAM_RST_N), U2.P1 (RESET_n)
- net GND: now also U2.B2 (VSS), U2.B3 (VDD), U2.B9 (VDD), U2.D1 (VDD), U2.E1 (VSS), U2.E9 (VSS), U2.G7 (VDD), U2.G8 (VSS), U2.J1 (VDD), U2.J9 (VDD), U2.K1 (VSS), U2.K9 (VSS), U2.L1 (VDD), U2.L9 (VDD), U2.M9 (VSS), U2.N1 (VSS), U2.R1 (VDD), U2.T1 (VSS), U2.T9 (VDD)
- new net +1V2: U2.A1 (VDDQ), U2.A2 (VSSQ), U2.A8 (VSSQ), U2.A9 (VDDQ), U2.C1 (VDDQ), U2.C9 (VSSQ), U2.D2 (VSSQ), U2.D8 (VSSQ), U2.D9 (VDDQ), U2.E3 (VSSQ), U2.E8 (VSSQ), U2.F1 (VSSQ), U2.F2 (VDDQ), U2.F8 (VDDQ), U2.G1 (VDDQ), U2.G9 (VDDQ), U2.H1 (VSSQ), U2.H9 (VSSQ), U2.J2 (VDDQ), U2.J8 (VDDQ)
- new net DDR_A15: U1.AA16 (PS_DDR_A15), U2.M8 (CAS_n/A15)
- new net DDR_A16: U1.Y16 (PS_DDR_A16), U2.L8 (RAS_n/A16)
- new net DDR_ACTN: U1.U15 (PS_DDR_ACT_N), U2.L3 (ACT_n)
- new net DDR_ALERTN: U1.T21 (PS_DDR_ALERT_N), U2.P9 (ALERT_n)
- new net DDR_PARITY: U1.U19 (PS_DDR_PARITY), U2.T3 (PAR)
- no-connect marks 2 -> 1
Other:
- note removed: "MT41K256M16TW-107:P x2\n"
- note removed: "XC7Z010"

Commit message: upd
Parts:
- added C?: 100nF, Capacitor_SMD:C_0805_2012Metric, symbol Device:C
- added R? (x2): 240, Resistor_SMD:R_0805_2012Metric, symbol Device:R
- added R?: 300, Resistor_SMD:R_0805_2012Metric, symbol Device:R
- added R?: 1K, Resistor_SMD:R_0805_2012Metric, symbol Device:R
Connections:
- net GND: now also U2.N9 (TEN), C?.1, R?.1, R?.2, R?.2
- net DDR_DQS_N1: now reaches U1.AA13 (PS_DDR_DQS_N1)
- net DDR_DQS_N1: now also U2.A7 (UDQS_c)
- net DDR_DQS_N0: now reaches U1.AA9 (PS_DDR_DQS_N0)
- net DDR_DQS_N0: now also U2.F3 (LDQS_c)
- net DDR_DM1: now reaches U1.AB14 (PS_DDR_DM1)
- net DDR_DM1: now also U2.E2 (NF/UDM_n/UDBI_n)
- net DDR_DM0: now reaches U1.AB9 (PS_DDR_DM0)
- net DDR_DM0: now also U2.E7 (NF/UDM_n/LDBI_n)
- net at U1.T19 (PS_DDR_ZQ): now also R?.1
- net DDR_BG0: now reaches U1.U16 (PS_DDR_BG0)
- net DDR_BG0: now also U2.M2 (BG0)
- net DDR_BA0: now reaches U1.U17 (PS_DDR_BA0)
- net DDR_BA0: now also U2.N2 (BA0)
- net DDR_CKE: now reaches U1.U22 (PS_DDR_CKE0)
- net DDR_CKE: now also U2.K2 (CKE)
- net DDR_BA1: now reaches U1.V17 (PS_DDR_BA1)
- net DDR_BA1: now also U2.N8 (BA1)
- net DDR_CK: now reaches U1.V20 (PS_DDR_CK0)
- net DDR_CK: now also U2.K7 (CK_t)
- net DDR_CS: now reaches U1.V22 (PS_DDR_CS_N0)
- net DDR_CS: now also U2.L7 (CS_n)
- net DDR_CK_N: now reaches U1.W20 (PS_DDR_CK_N0)
- net DDR_CK_N: now also U2.K8 (CK_c)
- net DDR_ODT: now reaches U1.W22 (PS_DDR_ODT0)
- net DDR_ODT: now also U2.K3 (ODT)
- net DDR_DQS_P1: now reaches U1.Y13 (PS_DDR_DQS_P1)
- net DDR_DQS_P1: now also U2.B7 (UDQS_t)
- net DDR_DQS_P0: now reaches U1.Y9 (PS_DDR_DQS_P0)
- net DDR_DQS_P0: now also U2.G3 (LDQS_t)
- net +2V5: now reaches U2.B1 (VPP)
- net +2V5: now also U2.R9 (VPP), R?.1, R?.2
- net at U2.F9 (ZQ): now also R?.1
- net at U2.M1 (VREFCA): now also C?.2
- new net +3V3: R?.2
- no-connect marks 1 -> 40

Commit message: upd
Parts:
- gave numbers to parts that had none: 5
Changed lines of the file:
@@
 	5650 6950 6150 6950
 $Comp
-L Device:R R?
+L Device:R R66
 U 1 1 601DA97F
 P 4200 7300
-F 0 "R?" V 4100 7150 50  0000 C CNN
+F 0 "R66" V 4100 7150 50  0000 C CNN
 F 1 "240" V 4100 7400 50  0000 C CNN
 F 2 "Resistor_SMD:R_0805_2012Metric" V 4130 7300 50  0001 C CNN
@@
 	4350 7300 4450 7300
 $Comp
-L power:GND #PWR?
+L power:GND #PWR0250
 U 1 1 601F2251
 P 3950 7300
-F 0 "#PWR?" H 3950 7050 50  0001 C CNN
+F 0 "#PWR0250" H 3950 7050 50  0001 C CNN
 F 1 "GND" V 3955 7172 50  0000 R CNN
 F 2 "" H 3950 7300 50  0001 C CNN
@@
 	3950 7300 4000 7300
 $Comp
-L power:GND #PWR?
+L power:GND #PWR0251
 U 1 1 601FE5C0
 P 4350 7100
-F 0 "#PWR?" H 4350 6850 50  0001 C CNN
+F 0 "#PWR0251" H 4350 6850 50  0001 C CNN
 F 1 "GND" V 4355 6972 50  0000 R CNN
 F 2 "" H 4350 7100 50  0001 C CNN
@@
 	4000 7300 4050 7300
 $Comp
-L Device:C C?
+L Device:C C37
 U 1 1 602CB8FE
 P 4250 7450
-F 0 "C?" V 4150 7600 50  0000 C CNN
+F 0 "C37" V 4150 7600 50  0000 C CNN
 F 1 "100nF" V 4150 7350 50  0000 C CNN
 F 2 "Capacitor_SMD:C_0805_2012Metric" H 4288 7300 50  0001 C CNN
@@
 	3950 6650 4450 6650
 $Comp
-L Device:R R?
+L Device:R R64
 U 1 1 6033A0AB
 P 2900 9350
-F 0 "R?" V 2693 9350 50  0000 C CNN
+F 0 "R64" V 2693 9350 50  0000 C CNN
 F 1 "300" V 2784 9350 50  0000 C CNN
 F 2 "Resistor_SMD:R_0805_2012Metric" V 2830 9350 50  0001 C CNN
@@
 $EndComp
 $Comp
-L Device:R R?
+L Device:R R65
 U 1 1 6033ABD1
 P 3350 9650
-F 0 "R?" H 3280 9604 50  0000 R CNN
+F 0 "R65" H 3280 9604 50  0000 R CNN
 F 1 "1K" H 3280 9695 50  0000 R CNN
 F 2 "Resistor_SMD:R_0805_2012Metric" V 3280 9650 50  0001 C CNN
@@
 	3350 9350 3350 9500
 $Comp
-L power:+3.3V #PWR?
+L power:+3.3V #PWR0252
 U 1 1 603A8B4A
 P 2350 9300
-F 0 "#PWR?" H 2350 9150 50  0001 C CNN
+F 0 "#PWR0252" H 2350 9150 50  0001 C CNN
 F 1 "+3.3V" H 2365 9473 50  0000 C CNN
 F 2 "" H 2350 9300 50  0001 C CNN
@@
 	2350 9350 2750 9350
 $Comp
-L power:GND #PWR?
+L power:GND #PWR0253
 U 1 1 603B7C6A
 P 3350 9950
-F 0 "#PWR?" H 3350 9700 50  0001 C CNN
+F 0 "#PWR0253" H 3350 9700 50  0001 C CNN
 F 1 "GND" H 3355 9777 50  0000 C CNN
 F 2 "" H 3350 9950 50  0001 C CNN
@@
 	3350 9950 3350 9800
 $Comp
-L power:+2V5 #PWR?
+L power:+2V5 #PWR0254
 U 1 1 603C73CB
 P 3650 9300
-F 0 "#PWR?" H 3650 9150 50  0001 C CNN
+F 0 "#PWR0254" H 3650 9150 50  0001 C CNN
 F 1 "+2V5" H 3665 9473 50  0000 C CNN
 F 2 "" H 3650 9300 50  0001 C CNN
@@
 	3350 9350 3650 9350
 $Comp
-L power:+2V5 #PWR?
+L power:+2V5 #PWR0255
 U 1 1 603F38FD
 P 3800 4050
-F 0 "#PWR?" H 3800 3900 50  0001 C CNN
+F 0 "#PWR0255" H 3800 3900 50  0001 C CNN
 F 1 "+2V5" V 3815 4178 50  0000 L CNN
 F 2 "" H 3800 4050 50  0001 C CNN
@@
 NoConn ~ 12150 6850
 $Comp
-L Device:R R?
+L Device:R R67
 U 1 1 60452FD6
 P 11650 8200
-F 0 "R?" H 11550 8150 50  0000 C CNN
+F 0 "R67" H 11550 8150 50  0000 C CNN
 F 1 "240" H 11800 8150 50  0000 C CNN
 F 2 "Resistor_SMD:R_0805_2012Metric" V 11580 8200 50  0001 C CNN
@@
 $EndComp
 $Comp
-L power:GND #PWR?
+L power:GND #PWR0256
 U 1 1 60452FDC
 P 11650 8450
-F 0 "#PWR?" H 11650 8200 50  0001 C CNN
+F 0 "#PWR0256" H 11650 8200 50  0001 C CNN
 F 1 "GND" V 11655 8322 50  0000 R CNN
 F 2 "" H 11650 8450 50  0001 C CNN

Commit message: upd
Parts:
- added C?: 100nF, Capacitor_SMD:C_0805_2012Metric, symbol Device:C
- added R?: 240, Resistor_SMD:R_0805_2012Metric, symbol Device:R
- added R? (x32): 15, symbol Zynq_UltraScale:R
- added U?: MT40A512M16, Zynq-eame_UltraScale_0:FBGA96_LY, symbol Zynq_UltraScale:MT40A512M16
Connections:
- net +1V2: now also U2.B3 (VDD), U2.B9 (VDD), U2.D1 (VDD), U2.G7 (VDD), U2.J1 (VDD), U2.J9 (VDD), U2.L1 (VDD), U2.L9 (VDD), U2.R1 (VDD), U2.T9 (VDD), U?.A1 (VDDQ), U?.A9 (VDDQ), U?.B3 (VDD), U?.B9 (VDD), U?.C1 (VDDQ), U?.D1 (VDD), U?.D9 (VDDQ), U?.F2 (VDDQ), U?.F8 (VDDQ), U?.G1 (VDDQ), U?.G7 (VDD), U?.G9 (VDDQ), U?.J1 (VDD), U?.J2 (VDDQ), U?.J8 (VDDQ), U?.J9 (VDD), U?.L1 (VDD), U?.L9 (VDD), U?.R1 (VDD), U?.T9 (VDD); no longer U2.A2 (VSSQ), U2.A8 (VSSQ), U2.C9 (VSSQ), U2.D2 (VSSQ), U2.D8 (VSSQ), U2.E3 (VSSQ), U2.E8 (VSSQ), U2.F1 (VSSQ), U2.H1 (VSSQ), U2.H9 (VSSQ)
- net +2V5: now also U?.B1 (VPP), U?.R9 (VPP)
- net DDR_A0: now also U?.P3 (A0)
- net DDR_A1: now also U?.P7 (A1)
- net DDR_A10: now also U?.M3 (A10/AP)
- net DDR_A11: now also U?.T2 (A11)
- net DDR_A12: now also U?.M7 (A12/BC_n)
- net DDR_A13: now also U?.T8 (A13)
- net DDR_A14: now also U?.L2 (WE_n/A14)
- net DDR_A15: now also U?.M8 (CAS_n/A15)
- net DDR_A16: now also U?.L8 (RAS_n/A16)
- net DDR_A2: now also U?.R3 (A2)
- net DDR_A3: now also U?.N7 (A3)
- net DDR_A4: now also U?.N3 (A4)
- net DDR_A5: now also U?.P8 (A5)
- net DDR_A6: now also U?.P2 (A6)
- net DDR_A7: now also U?.R8 (A7)
- net DDR_A8: now also U?.R2 (A8)
- net DDR_A9: now also U?.R7 (A9)
- net DDR_ACTN: now also U?.L3 (ACT_n)
- net DDR_ALERTN: now also U?.P9 (ALERT_n)
- net DDR_BA0: now also U?.N2 (BA0)
- net DDR_BA1: now also U?.N8 (BA1)
- net DDR_BG0: now also U?.M2 (BG0)
- net DDR_CK: now also U?.K7 (CK_t)
- net DDR_CKE: now also U?.K2 (CKE)
- net DDR_CK_N: now also U?.K8 (CK_c)
- net DDR_CS: now also U?.L7 (CS_n)
- net DDR_D0: now also R?.2; no longer U1.AB11 (PS_DDR_DQ0)
- net DDR_D1: now also R?.2; no longer U1.Y10 (PS_DDR_DQ1)
- net DDR_D10: now also R?.2; no longer U1.AA12 (PS_DDR_DQ10)
- net DDR_D11: now also R?.2; no longer U1.AB12 (PS_DDR_DQ11)
- net DDR_D12: now also R?.2; no longer U1.Y14 (PS_DDR_DQ12)
- net DDR_D13: now also R?.2; no longer U1.AA14 (PS_DDR_DQ13)
- net DDR_D14: now also R?.2; no longer U1.Y15 (PS_DDR_DQ14)
- net DDR_D15: now also R?.2; no longer U1.AB15 (PS_DDR_DQ15)
- net DDR_D2: now also R?.2; no longer U1.AB10 (PS_DDR_DQ2)
- net DDR_D3: now also R?.2; no longer U1.W10 (PS_DDR_DQ3)
- net DDR_D4: now also R?.2; no longer U1.AA8 (PS_DDR_DQ4)
- net DDR_D5: now also R?.2; no longer U1.Y8 (PS_DDR_DQ5)
- net DDR_D6: now also R?.2; no longer U1.AB7 (PS_DDR_DQ6)
- net DDR_D7: now also R?.2; no longer U1.AA7 (PS_DDR_DQ7)
- net DDR_D8: now also R?.2; no longer U1.AA11 (PS_DDR_DQ8)
- net DDR_D9: now also R?.2; no longer U1.Y11 (PS_DDR_DQ9)
- net DDR_DM0: now also U1.U9 (PS_DDR_DM2)
- net DDR_DM1: now also U1.W13 (PS_DDR_DM3)
- net DDR_ODT: now also U?.K3 (ODT)
- net DDR_PARITY: now also U?.T3 (PAR)
- net DDR_RESETN: now also U?.P1 (RESET_n)
- net GND: now also U2.A2 (VSSQ), U2.A8 (VSSQ), U2.C9 (VSSQ), U2.D2 (VSSQ), U2.D8 (VSSQ), U2.E3 (VSSQ), U2.E8 (VSSQ), U2.F1 (VSSQ), U2.H1 (VSSQ), U2.H9 (VSSQ), C?.1, R?.2, U?.A2 (VSSQ), U?.A8 (VSSQ), U?.B2 (VSS), U?.C9 (VSSQ), U?.D2 (VSSQ), U?.D8 (VSSQ), U?.E1 (VSS), U?.E3 (VSSQ), U?.E8 (VSSQ), U?.E9 (VSS), U?.F1 (VSSQ), U?.G8 (VSS), U?.H1 (VSSQ), U?.H9 (VSSQ), U?.K1 (VSS), U?.K9 (VSS), U?.M9 (VSS), U?.N1 (VSS), U?.N9 (TEN), U?.T1 (VSS); no longer U2.B3 (VDD), U2.B9 (VDD), U2.D1 (VDD), U2.G7 (VDD), U2.J1 (VDD), U2.J9 (VDD), U2.L1 (VDD), U2.L9 (VDD), U2.R1 (VDD), U2.T9 (VDD)
- net at U1.T10 (PS_DDR_DQ23): now also R?.1
- net at U1.T9 (PS_DDR_DQ21): now also R?.1
- net at U1.U10 (PS_DDR_DQ22): now also R?.1
- net at U1.U11 (PS_DDR_DQ24): now also R?.1
- net at U1.U12 (PS_DDR_DQ25): now also R?.1
- net at U1.U14 (PS_DDR_DQ29): now also R?.1
- net at U1.U7 (PS_DDR_DQ20): now also R?.1
- net at U1.V10 (PS_DDR_DQ19): now also R?.1
- net DDR_DQS_P3: now reaches U1.V12 (PS_DDR_DQS_P3)
- net DDR_DQS_P3: now also U?.B7 (UDQS_t)
- net DDR_DQS_N3: now reaches U1.V13 (PS_DDR_DQS_N3)
- net DDR_DQS_N3: now also U?.A7 (UDQS_c)
- net at U1.V14 (PS_DDR_DQ28): now also R?.1
- net at U1.V15 (PS_DDR_DQ31): now also R?.1
- net at U1.V7 (PS_DDR_DQ18): now also R?.1
- net DDR_DQS_N2: now reaches U1.V8 (PS_DDR_DQS_N2)
- net DDR_DQS_N2: now also U?.F3 (LDQS_c)
- net DDR_DQS_P2: now reaches U1.V9 (PS_DDR_DQS_P2)
- net DDR_DQS_P2: now also U?.G3 (LDQS_t)
- net at U1.W11 (PS_DDR_DQ27): now also R?.1
- net at U1.W12 (PS_DDR_DQ26): now also R?.1
- net at U1.W15 (PS_DDR_DQ30): now also R?.1
- net at U1.W7 (PS_DDR_DQ17): now also R?.1
- net at U1.W8 (PS_DDR_DQ16): now also R?.1
- new net: R?.1, U1.AA11 (PS_DDR_DQ8)
- new net: R?.1, U1.AA12 (PS_DDR_DQ10)
- new net: R?.1, U1.AA14 (PS_DDR_DQ13)
- new net: R?.1, U1.AA7 (PS_DDR_DQ7)
- new net: R?.1, U1.AA8 (PS_DDR_DQ4)
- new net: R?.1, U1.AB10 (PS_DDR_DQ2)
- new net: R?.1, U1.AB11 (PS_DDR_DQ0)
- new net: R?.1, U1.AB12 (PS_DDR_DQ11)
- new net: R?.1, U1.AB15 (PS_DDR_DQ15)
- new net: R?.1, U1.AB7 (PS_DDR_DQ6)
- new net: R?.1, U1.W10 (PS_DDR_DQ3)
- new net: R?.1, U1.Y10 (PS_DDR_DQ1)
- new net: R?.1, U1.Y11 (PS_DDR_DQ9)
- new net: R?.1, U1.Y14 (PS_DDR_DQ12)
- new net: R?.1, U1.Y15 (PS_DDR_DQ14)
- new net: R?.1, U1.Y8 (PS_DDR_DQ5)
- new net: R?.1, U?.F9 (ZQ)
- new net: C?.2, U?.M1 (VREFCA)
- new net DDR_D16: R?.2, U?.G2 (DQ0)
- new net DDR_D17: R?.2, U?.F7 (DQ1)
- new net DDR_D18: R?.2, U?.H3 (DQ2)
- new net DDR_D19: R?.2, U?.H7 (DQ3)
- new net DDR_D20: R?.2, U?.H2 (DQ4)
- new net DDR_D21: R?.2, U?.H8 (DQ5)
- new net DDR_D22: R?.2, U?.J3 (DQ6)
- new net DDR_D23: R?.2, U?.J7 (DQ7)
- new net DDR_D24: R?.2, U?.A3 (DQ8)
- new net DDR_D25: R?.2, U?.B8 (DQ9)
- new net DDR_D26: R?.2, U?.C3 (DQ10)
- new net DDR_D27: R?.2, U?.C7 (DQ11)
- new net DDR_D28: R?.2, U?.C2 (DQ12)
- new net DDR_D29: R?.2, U?.C8 (DQ13)
- new net DDR_D30: R?.2, U?.D3 (DQ14)
- new net DDR_D31: R?.2, U?.D7 (DQ15)
- new net DDR_DM2: U?.E7 (NF/UDM_n/LDBI_n)
- new net DDR_DM3: U?.E2 (NF/UDM_n/UDBI_n)
- no-connect marks 40 -> 18
Other:
- moved on the sheet: C37, R66, U2
