File: Zynq-eame_0/KiCad/DDR.sch (KiCad schematic (older format))
At the start: 35 parts, among them U5 XC7Z010-BUENO, U6 MT41K256M16TW-107_P, U7 MT41K256M16TW-107_P

Commit message: uod
Parts:
- U5: symbol Zynq_7000:XC7Z010-BUENO -> Zynq-eame_0-rescue:XC7Z010-BUENO-Zynq_7000
- U6, U7: symbol Zynq_7000:MT41K256M16TW-107_P -> Zynq-eame_0-rescue:MT41K256M16TW-107_P-Zynq_7000
Changed lines of the file:
@@
 EESchema Schematic File Version 4
-LIBS:Zynq-eame_0-cache
 EELAYER 30 0
 EELAYER END
@@
 DDR_VREF
 $Comp
-L Zynq_7000:MT41K256M16TW-107_P U6
+L Zynq-eame_0-rescue:MT41K256M16TW-107_P-Zynq_7000 U6
 U 1 1 60150218
 P 3400 3800
@@
 	12000 1950 11400 1950
 $Comp
-L Zynq_7000:MT41K256M16TW-107_P U7
+L Zynq-eame_0-rescue:MT41K256M16TW-107_P-Zynq_7000 U7
 U 1 1 5FF224F6
 P 6750 3850
@@
 	14550 7200 15050 7200
 $Comp
-L Zynq_7000:XC7Z010-BUENO U5
+L Zynq-eame_0-rescue:XC7Z010-BUENO-Zynq_7000 U5
 U 5 1 601CE83E
 P 13500 5950
