File: Zynq-eame_0/KiCad/Zynq-eame_0.kicad_pcb (KiCad board)
At the start: 4 copper layers, 150 x 100 mm, 186 parts, among them J1 Conn_01x06, J2 USB_B_Micro, J3 Micro_SD_Card, J4 USB_B_Micro, J5 Barrel_Jack, J6 HDMI_A, Q1 MMBT3904, Q2 MMBT3904, Q3 MMBT3904, Q4 MMBT3904, Q5 MMBF170, Q6 MMBF170, Q7 MMBF170, Q8 MMBF170, Q9 MMBF170, U1 TPS563201, U10 PINES_ALIMENTACION, U11 FT2232H, U12 PINES_ALIMENTACION, U13 93C46, U14 S25FL128S, U2 TPS563201, U3 TPS563201, U4 TPS563201, U5 XC7Z010-BUENO, U6 MT41K256M16TW-107_P, U7 MT41K256M16TW-107_P, U8 CP2102N-A01-GQFN28, U9 TPS3106K33DBV, X1 ASE-33.333MHz, Y1 12MHz

Commit message: update
Parts:
- moved U10 2.09 mm to (166.4, 157.1)
- moved JP2 0.82 mm to (139.7, 158.8)
- moved JP1 0.80 mm to (265.9, 111.0)
- moved JP3 0.51 mm to (229.9, 68.8)
Routing:
- net GND: track 30.5 -> 47.9 mm
