File: Zynq-eame_0/KiCad/alimentaciones.sch (KiCad schematic (older format))
At the start: 54 parts, among them J5 Barrel_Jack, Q1 MMBT3904, Q2 MMBT3904, Q3 MMBT3904, Q4 MMBT3904, U1 TPS563201, U2 TPS563201, U3 TPS563201, U4 TPS563201, U5 XC7Z010-BUENO, U9 TPS3106K33DBV

Commit message: uod
Parts:
- U1, U2, U3, U4: symbol Zynq_7000:TPS563201 -> Zynq-eame_0-rescue:TPS563201-Zynq_7000
- U5: symbol Zynq_7000:XC7Z010-BUENO -> Zynq-eame_0-rescue:XC7Z010-BUENO-Zynq_7000
- U9: symbol Zynq_7000:TPS3106K33DBV -> Zynq-eame_0-rescue:TPS3106K33DBV-Zynq_7000
Changed lines of the file:
@@
 EESchema Schematic File Version 4
-LIBS:Zynq-eame_0-cache
 EELAYER 30 0
 EELAYER END
@@
 $EndDescr
 $Comp
-L Zynq_7000:TPS563201 U?
+L Zynq-eame_0-rescue:TPS563201-Zynq_7000 U?
 U 1 1 5FFEBF57
 P 3100 1900
@@
 $EndComp
 $Comp
-L Zynq_7000:VIN #PWR?
+L Zynq-eame_0-rescue:VIN-Zynq_7000 #PWR?
 U 1 1 5FFEBFD2
 P 1500 1650
@@
 	5250 1750 5400 1750
 $Comp
-L Zynq_7000:TPS563201 U?
+L Zynq-eame_0-rescue:TPS563201-Zynq_7000 U?
 U 1 1 5FFEBFDE
 P 3700 4100
@@
 	6000 4500 6000 4400
 $Comp
-L Zynq_7000:VIN #PWR?
+L Zynq-eame_0-rescue:VIN-Zynq_7000 #PWR?
 U 1 1 5FFEC04D
 P 1350 3850
@@
 	2750 5300 2750 4850
 $Comp
-L Zynq_7000:TPS563201 U?
+L Zynq-eame_0-rescue:TPS563201-Zynq_7000 U?
 U 1 1 5FFEC097
 P 3050 6500
@@
 	5350 6900 5350 6800
 $Comp
-L Zynq_7000:VIN #PWR?
+L Zynq-eame_0-rescue:VIN-Zynq_7000 #PWR?
 U 1 1 5FFEC100
 P 1450 6250
@@
 	3950 6850 4450 6850
 $Comp
-L Zynq_7000:TPS563201 U?
+L Zynq-eame_0-rescue:TPS563201-Zynq_7000 U?
 U 1 1 5FFEC122
 P 3400 8500
@@
 	5700 8900 5700 8800
 $Comp
-L Zynq_7000:VIN #PWR?
+L Zynq-eame_0-rescue:VIN-Zynq_7000 #PWR?
 U 1 1 5FFEC191
 P 900 8250
@@
 	6600 8500 6400 8500
 $Comp
-L Zynq_7000:VCCO_34 #PWR?
+L Zynq-eame_0-rescue:VCCO_34-Zynq_7000 #PWR?
 U 1 1 5FFEC1F6
 P 6600 8250
@@
 $EndComp
 $Comp
-L Zynq_7000:VCCO_34 #PWR044
+L Zynq-eame_0-rescue:VCCO_34-Zynq_7000 #PWR044
 U 1 1 60ADBC4F
 P 13400 6050
@@
 	13400 7250 13400 7350
 $Comp
-L Zynq_7000:XC7Z010-BUENO U5
+L Zynq-eame_0-rescue:XC7Z010-BUENO-Zynq_7000 U5
 U 8 1 6012E22C
 P 12350 7400
@@
 $EndComp
 $Comp
-L Zynq_7000:XC7Z010-BUENO U5
+L Zynq-eame_0-rescue:XC7Z010-BUENO-Zynq_7000 U5
 U 9 1 6013FBF4
 P 12400 2350
@@
 	8500 1400 8650 1400
 $Comp
-L Zynq_7000:VIN #PWR0176
+L Zynq-eame_0-rescue:VIN-Zynq_7000 #PWR0176
 U 1 1 6044FA90
 P 9200 1350
@@
 Voltage input\n\n
 $Comp
-L Zynq_7000:TPS3106K33DBV U9
+L Zynq-eame_0-rescue:TPS3106K33DBV-Zynq_7000 U9
 U 1 1 60DB874D
 P 8100 3350
