File: Zynq-eame_0/KiCad/ent_sal.sch (KiCad schematic (older format))
At the start: 52 parts, among them J6 HDMI_A, Q5 MMBF170, Q6 MMBF170, Q7 MMBF170, Q8 MMBF170, Q9 MMBF170, U10 PINES_ALIMENTACION, U12 PINES_ALIMENTACION, U5 XC7Z010-BUENO

Commit message: update
Changed lines of the file:
@@
 EESchema Schematic File Version 4
-LIBS:Diseno_1-cache
+LIBS:Zynq-eame_0-cache
 EELAYER 30 0
 EELAYER END
@@
 Wire Wire Line
 	12550 3300 12550 3150
-$Comp
-L Zynq_7000:TPD12S016 #U018
-U 1 1 606DDBF4
-P 12600 2350
-F 0 "#U018" H 12500 3650 50  0000 C CNN
-F 1 "TPD12S016" H 12500 3550 50  0000 C CNN
-F 2 "ZYNQ_7000:TSSOP-24-1_copy" H 12150 3200 50  0001 C CNN
-F 3 "https://www.ti.com/lit/ds/symlink/tpd12s016.pdf" H 12150 3200 50  0001 C CNN
-	1    12600 2350
-	1    0    0    -1
-$EndComp
 Wire Notes Line
 	10500 3750 10500 700
@@
 	0    -1   -1   0
 $EndComp
+$Comp
+L Zynq_7000:TPD12S016 #U0101
+U 1 1 60102532
+P 12600 2350
+F 0 "#U0101" H 12600 3665 50  0000 C CNN
+F 1 "TPD12S016" H 12600 3574 50  0000 C CNN
+F 2 "ZYNQ_7000:SOIC-24" H 11500 3150 50  0001 C CNN
+F 3 "https://www.ti.com/lit/ds/symlink/tpd12s016.pdf" H 11500 3150 50  0001 C CNN
+	1    12600 2350
+	1    0    0    -1
+$EndComp
 $EndSCHEMATC

Commit message: uod
Parts:
- JP1: symbol Zynq_7000:PINES_48 -> Zynq-eame_0-rescue:PINES_48-Zynq_7000
- JP2: symbol Zynq_7000:PIN_25 -> Zynq-eame_0-rescue:PIN_25-Zynq_7000
- JP3: symbol Zynq_7000:PINES_38 -> Zynq-eame_0-rescue:PINES_38-Zynq_7000
- U10, U12: symbol Zynq_7000:PINES_ALIMENTACION -> Zynq-eame_0-rescue:PINES_ALIMENTACION-Zynq_7000
- U5: symbol Zynq_7000:XC7Z010-BUENO -> Zynq-eame_0-rescue:XC7Z010-BUENO-Zynq_7000
Changed lines of the file:
@@
 EESchema Schematic File Version 4
-LIBS:Zynq-eame_0-cache
 EELAYER 30 0
 EELAYER END
@@
 $EndDescr
 $Comp
-L Zynq_7000:XC7Z010-BUENO U5
+L Zynq-eame_0-rescue:XC7Z010-BUENO-Zynq_7000 U5
 U 3 1 5FE9FB12
 P 2050 7850
@@
 $EndComp
 $Comp
-L Zynq_7000:XC7Z010-BUENO U5
+L Zynq-eame_0-rescue:XC7Z010-BUENO-Zynq_7000 U5
 U 4 1 5FEA9F18
 P 5400 7550
@@
 	11250 2750 11900 2750
 $Comp
-L Zynq_7000:VIN #PWR0178
+L Zynq-eame_0-rescue:VIN-Zynq_7000 #PWR0178
 U 1 1 6014D0BB
 P 11350 2850
@@
 HDMI\n
 $Comp
-L Zynq_7000:PINES_ALIMENTACION U10
+L Zynq-eame_0-rescue:PINES_ALIMENTACION-Zynq_7000 U10
 U 1 1 600B2403
 P 3850 1450
@@
 $EndComp
 $Comp
-L Zynq_7000:PINES_ALIMENTACION U12
+L Zynq-eame_0-rescue:PINES_ALIMENTACION-Zynq_7000 U12
 U 1 1 6013B241
 P 3850 2600
@@
 	3750 2250 4400 2250
 $Comp
-L Zynq_7000:VIN #PWR0196
+L Zynq-eame_0-rescue:VIN-Zynq_7000 #PWR0196
 U 1 1 604043AB
 P 4000 1900
@@
 Connection ~ 4000 1850
 $Comp
-L Zynq_7000:VIN #PWR0197
+L Zynq-eame_0-rescue:VIN-Zynq_7000 #PWR0197
 U 1 1 6044884E
 P 4000 3050
@@
 NoConn ~ 2800 10200
 $Comp
-L Zynq_7000:PINES_48 JP1
+L Zynq-eame_0-rescue:PINES_48-Zynq_7000 JP1
 U 1 1 6211BC63
 P 1750 2250
@@
 	7650 4600 15950 4600
 $Comp
-L Zynq_7000:PIN_25 JP2
+L Zynq-eame_0-rescue:PIN_25-Zynq_7000 JP2
 U 1 1 6138B5D5
 P 5900 1850
@@
 	6500 2400 6300 2400
 $Comp
-L Zynq_7000:PINES_38 JP3
+L Zynq-eame_0-rescue:PINES_38-Zynq_7000 JP3
 U 1 1 61537FB4
 P 8250 2050
@@
 $EndComp
 $Comp
-L Zynq_7000:TPD12S016 #U0101
+L Zynq-eame_0-rescue:TPD12S016-Zynq_7000 #U0101
 U 1 1 60102532
 P 12600 2350
