File: Zynq-eame_0/KiCad/referencia.sch (KiCad schematic (older format))
At the start: 50 parts, among them J1 Conn_01x06, J2 USB_B_Micro, J3 Micro_SD_Card, J4 USB_B_Micro, U11 FT2232H, U13 93C46, U14 S25FL128S, U5 XC7Z010-BUENO, U8 CP2102N-A01-GQFN28, X1 ASE-33.333MHz, Y1 12MHz

Commit message: update
Parts:
- C46, C47, C48, C49, C50, C51, C52: value C -> 100nF
Changed lines of the file:
@@
 EESchema Schematic File Version 4
-LIBS:Diseno_1-cache
+LIBS:Zynq-eame_0-cache
 EELAYER 30 0
 EELAYER END
@@
 P 6200 5950
 F 0 "C46" H 6315 5996 50  0000 L CNN
-F 1 "C" H 6315 5905 50  0000 L CNN
+F 1 "100nF" H 6250 5850 50  0000 L CNN
 F 2 "Capacitor_SMD:C_0805_2012Metric" H 6238 5800 50  0001 C CNN
 F 3 "~" H 6200 5950 50  0001 C CNN
@@
 P 6550 5950
 F 0 "C47" H 6665 5996 50  0000 L CNN
-F 1 "C" H 6665 5905 50  0000 L CNN
+F 1 "100nF" H 6600 5850 50  0000 L CNN
 F 2 "Capacitor_SMD:C_0805_2012Metric" H 6588 5800 50  0001 C CNN
 F 3 "~" H 6550 5950 50  0001 C CNN
@@
 P 6900 5950
 F 0 "C48" H 7015 5996 50  0000 L CNN
-F 1 "C" H 7015 5905 50  0000 L CNN
+F 1 "100nF" H 6950 5850 50  0000 L CNN
 F 2 "Capacitor_SMD:C_0805_2012Metric" H 6938 5800 50  0001 C CNN
 F 3 "~" H 6900 5950 50  0001 C CNN
@@
 P 7200 5950
 F 0 "C49" H 7315 5996 50  0000 L CNN
-F 1 "C" H 7315 5905 50  0000 L CNN
+F 1 "100nF" H 7250 5850 50  0000 L CNN
 F 2 "Capacitor_SMD:C_0805_2012Metric" H 7238 5800 50  0001 C CNN
 F 3 "~" H 7200 5950 50  0001 C CNN
@@
 P 7500 5950
 F 0 "C50" H 7615 5996 50  0000 L CNN
-F 1 "C" H 7615 5905 50  0000 L CNN
+F 1 "100nF" H 7550 5850 50  0000 L CNN
 F 2 "Capacitor_SMD:C_0805_2012Metric" H 7538 5800 50  0001 C CNN
 F 3 "~" H 7500 5950 50  0001 C CNN
@@
 P 7800 5950
 F 0 "C51" H 7915 5996 50  0000 L CNN
-F 1 "C" H 7915 5905 50  0000 L CNN
+F 1 "100nF" H 7850 5850 50  0000 L CNN
 F 2 "Capacitor_SMD:C_0805_2012Metric" H 7838 5800 50  0001 C CNN
 F 3 "~" H 7800 5950 50  0001 C CNN
@@
 P 8100 5950
 F 0 "C52" H 8215 5996 50  0000 L CNN
-F 1 "C" H 8215 5905 50  0000 L CNN
+F 1 "100nF" H 8150 5850 50  0000 L CNN
 F 2 "Capacitor_SMD:C_0805_2012Metric" H 8138 5800 50  0001 C CNN
 F 3 "~" H 8100 5950 50  0001 C CNN

Commit message: uod
Parts:
- J2, J4: symbol Connector:USB_B_Micro -> Zynq-eame_0-rescue:USB_B_Micro-Connector
- U11: symbol Interface_USB:FT2232H -> Zynq-eame_0-rescue:FT2232H-Interface_USB
- U13: symbol Zynq_7000:93C46 -> Zynq-eame_0-rescue:93C46-Zynq_7000
- U14: symbol Zynq_7000:S25FL128S -> Zynq-eame_0-rescue:S25FL128S-Zynq_7000
- U5: symbol Zynq_7000:XC7Z010-BUENO -> Zynq-eame_0-rescue:XC7Z010-BUENO-Zynq_7000
Changed lines of the file:
@@
 EESchema Schematic File Version 4
-LIBS:Zynq-eame_0-cache
 EELAYER 30 0
 EELAYER END
@@
 $EndDescr
 $Comp
-L Zynq_7000:XC7Z010-BUENO U5
+L Zynq-eame_0-rescue:XC7Z010-BUENO-Zynq_7000 U5
 U 2 1 6015CDE4
 P 12200 6050
@@
 $EndComp
 $Comp
-L Zynq_7000:XC7Z010-BUENO U5
+L Zynq-eame_0-rescue:XC7Z010-BUENO-Zynq_7000 U5
 U 6 1 601651B9
 P 12300 2500
@@
 $EndComp
 $Comp
-L Zynq_7000:XC7Z010-BUENO U5
+L Zynq-eame_0-rescue:XC7Z010-BUENO-Zynq_7000 U5
 U 7 1 6016DBA7
 P 14350 4350
@@
 $EndComp
 $Comp
-L Zynq_7000:XC7Z010-BUENO U5
+L Zynq-eame_0-rescue:XC7Z010-BUENO-Zynq_7000 U5
 U 1 1 6017695E
 P 14300 9300
@@
 	14900 8600 15200 8600
 $Comp
-L Connector:USB_B_Micro J2
+L Zynq-eame_0-rescue:USB_B_Micro-Connector J2
 U 1 1 5FF0ED8B
 P 1700 8400
@@
 	14900 5550 15350 5550
 $Comp
-L Interface_USB:FT2232H U11
+L Zynq-eame_0-rescue:FT2232H-Interface_USB U11
 U 1 1 600AACC3
 P 4600 3900
@@
 Connection ~ 4000 6250
 $Comp
-L Connector:USB_B_Micro J4
+L Zynq-eame_0-rescue:USB_B_Micro-Connector J4
 U 1 1 601ABA7F
 P 1000 3100
@@
 MIO, JTAG & REFERENCE\n
 $Comp
-L Zynq_7000:93C46 U13
+L Zynq-eame_0-rescue:93C46-Zynq_7000 U13
 U 1 1 6015CC72
 P 1550 5250
@@
 	11050 9350 11050 9450
 $Comp
-L Zynq_7000:S25FL128S U14
+L Zynq-eame_0-rescue:S25FL128S-Zynq_7000 U14
 U 1 1 60068CB9
 P 9850 2350
